File: kicad_files/PAM8403DR-H.kicad_sch (KiCad schematic)
At the start: 19 parts, among them J1 INL, J2 INR, J3 ~{SHDN}, J4 ~{MUTE}, J5 LOUT+, J6 LOUT-, J7 ROUT-, J8 ROUT+, U1 PAM8403D

Commit message: routing completed
Parts:
- added J10: GND, Connector_PinHeader_1.27mm:PinHeader_1x01_P1.27mm_Vertical, symbol Connector:Conn_01x01_Male
- added J9: 5V, Connector_PinHeader_1.27mm:PinHeader_1x01_P1.27mm_Vertical, symbol Connector:Conn_01x01_Male
Connections:
- net +5V: now also J9.1 (Pin_1)
- net GND: now also J10.1 (Pin_1)
Changed lines of the file:
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@@
+    (stroke (width 0) (type default) (color 0 0 0 0))
+  )
+  (wire (pts (xy 107.95 59.69) (xy 107.95 56.515))
     (stroke (width 0) (type default) (color 0 0 0 0))
   )
@@
     (stroke (width 0) (type default) (color 0 0 0 0))
   )
+  (wire (pts (xy 107.95 66.675) (xy 107.95 69.85))
+    (stroke (width 0) (type default) (color 0 0 0 0))
+  )
   (wire (pts (xy 240.665 95.25) (xy 248.92 95.25))
     (stroke (width 0) (type default) (color 0 0 0 0))
@@
   )
   (wire (pts (xy 124.46 97.155) (xy 138.43 97.155))
+    (stroke (width 0) (type default) (color 0 0 0 0))
+  )
+  (wire (pts (xy 103.505 59.69) (xy 107.95 59.69))
+    (stroke (width 0) (type default) (color 0 0 0 0))
+  )
+  (wire (pts (xy 103.505 66.675) (xy 107.95 66.675))
     (stroke (width 0) (type default) (color 0 0 0 0))
   )
@@
       (effects (font (size 1.27 1.27)) (justify left) hide)
     )
+  )
+  (symbol (lib_id "power:GND") (at 107.95 69.85 0) (unit 1)
+    (in_bom yes) (on_board yes) (fields_autoplaced)
+    (property "Reference" "#PWR06" (id 0) (at 107.95 76.2 0)
+      (effects (font (size 1.27 1.27)) hide)
+    )
+    (property "Value" "GND" (id 1) (at 107.95 74.295 0))
+    (property "Footprint" "" (id 2) (at 107.95 69.85 0)
+      (effects (font (size 1.27 1.27)) hide)
+    )
+    (property "Datasheet" "" (id 3) (at 107.95 69.85 0)
+      (effects (font (size 1.27 1.27)) hide)
+    )
+    (pin "1")
   )
   (symbol (lib_id "Device:R_Small") (at 140.97 89.535 90) (unit 1)
@@
     )
     (property "Datasheet" "~" (id 3) (at 43.18 87.63 0)
+      (effects (font (size 1.27 1.27)) hide)
+    )
+    (pin "1")
+  )
+  (symbol (lib_id "Connector:Conn_01x01_Male") (at 98.425 59.69 0) (unit 1)
+    (in_bom yes) (on_board yes)
+    (property "Reference" "J9" (id 0) (at 99.06 55.245 0))
+    (property "Value" "5V" (id 1) (at 99.06 57.785 0))
+    (property "Footprint" "Connector_PinHeader_1.27mm:PinHeader_1x01_P1.27mm_Vertical" (id 2) (at 98.425 59.69 0)
+      (effects (font (size 1.27 1.27)) hide)
+    )
+    (property "Datasheet" "~" (id 3) (at 98.425 59.69 0)
       (effects (font (size 1.27 1.27)) hide)
     )
@@
     (pin "1")
   )
+  (symbol (lib_id "power:+5V") (at 107.95 56.515 0) (unit 1)
+    (in_bom yes) (on_board yes) (fields_autoplaced)
+    (property "Reference" "#PWR05" (id 0) (at 107.95 60.325 0)
+      (effects (font (size 1.27 1.27)) hide)
+    )
+    (property "Value" "+5V" (id 1) (at 107.95 51.435 0))
+    (property "Footprint" "" (id 2) (at 107.95 56.515 0)
+      (effects (font (size 1.27 1.27)) hide)
+    )
+    (property "Datasheet" "" (id 3) (at 107.95 56.515 0)
+      (effects (font (size 1.27 1.27)) hide)
+    )
+    (pin "1")
+  )
   (symbol (lib_id "Device:C_Small") (at 133.35 89.535 90) (unit 1)
     (in_bom yes) (on_board yes)
@@
     (pin "1")
     (pin "2")
+  )
+  (symbol (lib_id "Connector:Conn_01x01_Male") (at 98.425 66.675 0) (unit 1)
+    (in_bom yes) (on_board yes)
+    (property "Reference" "J10" (id 0) (at 99.06 61.595 0))
+    (property "Value" "GND" (id 1) (at 99.06 64.135 0))
+    (property "Footprint" "Connector_PinHeader_1.27mm:PinHeader_1x01_P1.27mm_Vertical" (id 2) (at 98.425 66.675 0)
+      (effects (font (size 1.27 1.27)) hide)
+    )
+    (property "Datasheet" "~" (id 3) (at 98.425 66.675 0)
+      (effects (font (size 1.27 1.27)) hide)
+    )
+    (pin "1")
   )
   (symbol (lib_id "power:+5V") (at 153.67 57.15 0) (unit 1)
@@
       (reference "#PWR04") (unit 1) (value "GND") (footprint "")
     )
+    (path "/d4f4e3a5-c34d-4e05-a13b-4c754f72711a"
+      (reference "#PWR05") (unit 1) (value "+5V") (footprint "")
+    )
+    (path "/0a5c73bb-eeaa-4d75-8541-c2f01166b2e6"
+      (reference "#PWR06") (unit 1) (value "GND") (footprint "")
+    )
     (path "/6f7102a2-8768-4a78-9930-71570ebc6e68"
       (reference "C1") (unit 1) (value "100nf") (footprint "Capacitor_SMD:C_0603_1608Metric_Pad1.08x0.95mm_HandSolder")
@@
       (reference "J8") (unit 1) (value "ROUT+") (footprint "Connector_PinHeader_1.27mm:PinHeader_1x01_P1.27mm_Vertical")
     )
+    (path "/45b6008f-81d4-4e4b-9225-4b5a490b0153"
+      (reference "J9") (unit 1) (value "5V") (footprint "Connector_PinHeader_1.27mm:PinHeader_1x01_P1.27mm_Vertical")
+    )
+    (path "/f21dcdbd-e148-4b2f-ae45-530ce8774095"
+      (reference "J10") (unit 1) (value "GND") (footprint "Connector_PinHeader_1.27mm:PinHeader_1x01_P1.27mm_Vertical")
+    )
     (path "/bf09237b-0f4b-4ff1-b6d9-ad42c02d8a02"
