File: kicad_files/BANK_14.kicad_sch (KiCad schematic)
At the start: 1 part, among them IC1 XC7S25-1CSGA225C

Commit message: schematic updated
Parts:
- added R20: 49.9, symbol Device:R_Small_US
Connections:
- net PIO31: now reaches IC1.J11 (IO_0_14)
- net PIO28: now reaches IC1.J15 (IO_L5P_T0_D06_14)
- net PIO27: now reaches IC1.K14 (IO_L4P_T0_D04_14)
- net UART_TXD_IN: now reaches IC1.K15 (IO_L5N_T0_D07_14)
- net UART_RXD_OUT: now reaches IC1.L12 (IO_L6N_T0_D08_VREF_14)
- net PIO29: now reaches IC1.L13 (IO_L7P_T1_D09_14)
- net PIO26: now reaches IC1.L14 (IO_L7N_T1_D10_14)
- net PIO23: now reaches IC1.L15 (IO_L4N_T0_D05_14)
- net GCLK: now reaches IC1.M9 (IO_L13P_T2_MRCC_14)
- net GCLK: now also R20.1
- no-connect marks 0 -> 2
Changed lines of the file:
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@@
 (kicad_sch (version 20230121) (generator eeschema)
   (paper "A4")
+  (no_connect (at 132.715 76.835))
+  (no_connect (at 132.715 64.135))
+  (wire (pts (xy 132.715 74.295) (xy 151.13 74.295))
+    (stroke (width 0) (type default))
+  )
+  (wire (pts (xy 132.715 61.595) (xy 151.13 61.595))
+    (stroke (width 0) (type default))
+  )
+  (wire (pts (xy 132.715 71.755) (xy 151.13 71.755))
+    (stroke (width 0) (type default))
+  )
+  (wire (pts (xy 132.715 69.215) (xy 151.13 69.215))
+    (stroke (width 0) (type default))
+  )
+  (wire (pts (xy 132.715 59.055) (xy 151.13 59.055))
+    (stroke (width 0) (type default))
+  )
+  (wire (pts (xy 132.715 56.515) (xy 151.13 56.515))
+    (stroke (width 0) (type default))
+  )
+  (wire (pts (xy 132.715 81.915) (xy 145.415 81.915))
+    (stroke (width 0) (type default))
+  )
+  (wire (pts (xy 132.715 66.675) (xy 151.13 66.675))
+    (stroke (width 0) (type default))
+  )
+  (wire (pts (xy 132.715 53.975) (xy 151.13 53.975))
+    (stroke (width 0) (type default))
+  )
+  (label "PIO29" (at 151.13 69.215 180) (fields_autoplaced)
+    (effects (font (size 1.27 1.27)) (justify right bottom))
+  )
+  (label "PIO23" (at 151.13 74.295 180) (fields_autoplaced)
+    (effects (font (size 1.27 1.27)) (justify right bottom))
+  )
+  (label "GCLK" (at 145.415 81.915 180) (fields_autoplaced)
+    (effects (font (size 1.27 1.27)) (justify right bottom))
+  )
+  (label "PIO27" (at 151.13 59.055 180) (fields_autoplaced)
+    (effects (font (size 1.27 1.27)) (justify right bottom))
+  )
+  (label "UART_RXD_OUT" (at 151.13 66.675 180) (fields_autoplaced)
+    (effects (font (size 1.27 1.27)) (justify right bottom))
+  )
+  (label "UART_TXD_IN" (at 151.13 61.595 180) (fields_autoplaced)
+    (effects (font (size 1.27 1.27)) (justify right bottom))
+  )
+  (label "PIO31" (at 151.13 53.975 180) (fields_autoplaced)
+    (effects (font (size 1.27 1.27)) (justify right bottom))
+  )
+  (label "PIO28" (at 151.13 56.515 180) (fields_autoplaced)
+    (effects (font (size 1.27 1.27)) (justify right bottom))
+  )
+  (label "PIO26" (at 151.13 71.755 180) (fields_autoplaced)
+    (effects (font (size 1.27 1.27)) (justify right bottom))
+  )
   (symbol (lib_id "SamacSys_Parts:XC7S25-1CSGA225C") (at 103.505 100.965 0) (unit 2)
     (in_bom yes) (on_board yes) (dnp no)
-    (property "Reference" "IC1" (at 103.505 24.13 0)
+    (property "Reference" "IC1" (at 100.965 43.18 0)
       (effects (font (size 1.27 1.27)))
     )
-    (property "Value" "XC7S25-1CSGA225C" (at 103.505 27.305 0)
+    (property "Value" "XC7S25-1CSGA225C" (at 100.965 46.355 0)
       (effects (font (size 1.27 1.27)))
     )
@@
     (pin "R1")
     (pin "R15")
-    (pin "E5")
-    (pin "F5")
-    (pin "G5")
-    (pin "G8")
-    (pin "G9")
-    (pin "H14")
-    (pin "H15")
-    (pin "H5")
-    (pin "H8")
-    (pin "H9")
     (pin "J11")
-    (pin "J12")
     (pin "J15")
-    (pin "J5")
-    (pin "J8")
-    (pin "J9")
-    (pin "K11")
-    (pin "K12")
-    (pin "K13")
     (pin "K14")
     (pin "K15")
-    (pin "K4")
-    (pin "K5")
     (pin "L10")
-    (pin "L11")
     (pin "L12")
     (pin "L13")
     (pin "L14")
     (pin "L15")
-    (pin "L4")
-    (pin "L5")
     (pin "M10")
     (pin "M13")
     (pin "M14")
     (pin "M15")
-    (pin "M5")
-    (pin "M6")
     (pin "M7")
     (pin "M8")
     (pin "M9")
-    (pin "N10")
-    (pin "N11")
     (pin "N12")
     (pin "N13")
     (pin "N14")
     (pin "N15")
-    (pin "N5")
     (pin "N6")
     (pin "N7")
     (pin "N8")
     (pin "N9")
-    (pin "P10")
     (pin "P11")
     (pin "P12")
@@
           (reference "IC1") (unit 2)
         )
+        (path "/94bd3a84-5526-4cf2-a5cc-3887356f447c/30d52c37-ae5c-405e-8a78-89b18a6efc4e/af489dd5-0e9e-4b3e-a401-f1288bd8b210"
+          (reference "IC1") (unit 2)
+        )
       )
+    )
+  )
+  (symbol (lib_id "Device:R_Small_US") (at 147.955 81.915 90) (unit 1)
+    (in_bom yes) (on_board yes) (dnp no)
+    (property "Reference" "R20" (at 147.955 80.01 90)
+      (effects (font (size 1.27 1.27)))
+    )
+    (property "Value" "49.9" (at 147.955 84.455 90)
+      (effects (font (size 1.27 1.27)))
+    )
+    (property "Footprint" "" (at 147.955 81.915 0)
+      (effects (font (size 1.27 1.27)) hide)
+    )
+    (property "Datasheet" "~" (at 147.955 81.915 0)
+      (effects (font (size 1.27 1.27)) hide)
+    )
+    (pin "1")
+    (pin "2")
+    (instances
+      (project "sparton_7"
+        (path "/94bd3a84-5526-4cf2-a5cc-3887356f447c/30d52c37-ae5c-405e-8a78-89b18a6efc4e/b9c5b3c3-3c31-4d87-a13a-ee1ac9be93fb"
+          (reference "R20") (unit 1)
+        )
+      )

Commit message: ftdi progess
Connections:
- net PIO30: now reaches IC1.M13 (IO_L8P_T1_D11_14)
- net PIO22: now reaches IC1.M14 (IO_L9P_T1_DQS_14)
- net PIO21: now reaches IC1.M15 (IO_L9N_T1_DQS_D13_14)
- net PIO18: now reaches IC1.N13 (IO_L8N_T1_D12_14)
- net PIO20: now reaches IC1.N14 (IO_L10P_T1_D14_14)
- net PIO19: now reaches IC1.N15 (IO_L10N_T1_D15_14)
- net PIO16: now reaches IC1.P14 (IO_L11P_T1_SRCC_14)
- net PIO17: now reaches IC1.P15 (IO_L11N_T1_SRCC_14)
- net USB_12MHZ: now reaches R20.2
- no-connect marks 2 -> 23
Changed lines of the file:
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@@
 (kicad_sch (version 20230121) (generator eeschema)
   (paper "A4")
+  (no_connect (at 132.715 97.155))
+  (no_connect (at 132.715 153.035))
   (no_connect (at 132.715 76.835))
+  (no_connect (at 132.715 109.855))
+  (no_connect (at 132.715 94.615))
+  (no_connect (at 132.715 79.375))
   (no_connect (at 132.715 64.135))
+  (no_connect (at 132.715 99.695))
+  (no_connect (at 132.715 155.575))
+  (no_connect (at 132.715 142.875))
+  (no_connect (at 132.715 127.635))
+  (no_connect (at 132.715 147.955))
+  (no_connect (at 132.715 140.335))
+  (no_connect (at 132.715 160.655))
+  (no_connect (at 132.715 122.555))
+  (no_connect (at 132.715 102.235))
+  (no_connect (at 132.715 84.455))
+  (no_connect (at 132.715 137.795))
+  (no_connect (at 132.715 145.415))
+  (no_connect (at 132.715 120.015))
+  (no_connect (at 132.715 130.175))
+  (no_connect (at 132.715 150.495))
+  (no_connect (at 132.715 158.115))
+  (wire (pts (xy 150.495 81.915) (xy 167.005 81.915))
+    (stroke (width 0) (type default))
+  )
+  (wire (pts (xy 132.715 89.535) (xy 151.13 89.535))
+    (stroke (width 0) (type default))
+  )
+  (wire (pts (xy 132.715 86.995) (xy 151.13 86.995))
+    (stroke (width 0) (type default))
+  )
   (wire (pts (xy 132.715 74.295) (xy 151.13 74.295))
     (stroke (width 0) (type default))
@@
     (stroke (width 0) (type default))
   )
+  (wire (pts (xy 132.715 132.715) (xy 151.13 132.715))
+    (stroke (width 0) (type default))
+  )
   (wire (pts (xy 132.715 59.055) (xy 151.13 59.055))
     (stroke (width 0) (type default))
@@
     (stroke (width 0) (type default))
   )
+  (wire (pts (xy 132.715 114.935) (xy 151.13 114.935))
+    (stroke (width 0) (type default))
+  )
+  (wire (pts (xy 132.715 112.395) (xy 151.13 112.395))
+    (stroke (width 0) (type default))
+  )
+  (wire (pts (xy 132.715 92.075) (xy 151.13 92.075))
+    (stroke (width 0) (type default))
+  )
+  (wire (pts (xy 132.715 135.255) (xy 151.13 135.255))
+    (stroke (width 0) (type default))
+  )
   (wire (pts (xy 132.715 81.915) (xy 145.415 81.915))
+    (stroke (width 0) (type default))
+  )
+  (wire (pts (xy 132.715 117.475) (xy 151.13 117.475))
     (stroke (width 0) (type default))
   )
@@
     (effects (font (size 1.27 1.27)) (justify right bottom))
   )
+  (label "PIO21" (at 151.13 92.075 180) (fields_autoplaced)
+    (effects (font (size 1.27 1.27)) (justify right bottom))
+  )
   (label "PIO23" (at 151.13 74.295 180) (fields_autoplaced)
+    (effects (font (size 1.27 1.27)) (justify right bottom))
+  )
+  (label "USB_12MHZ" (at 167.005 81.915 180) (fields_autoplaced)
+    (effects (font (size 1.27 1.27)) (justify right bottom))
+  )
+  (label "PIO20" (at 151.13 114.935 180) (fields_autoplaced)
+    (effects (font (size 1.27 1.27)) (justify right bottom))
+  )
+  (label "PIO30" (at 151.13 86.995 180) (fields_autoplaced)
     (effects (font (size 1.27 1.27)) (justify right bottom))
   )
@@
     (effects (font (size 1.27 1.27)) (justify right bottom))
   )
+  (label "PIO17" (at 151.13 135.255 180) (fields_autoplaced)
+    (effects (font (size 1.27 1.27)) (justify right bottom))
+  )
+  (label "PIO16" (at 151.13 132.715 180) (fields_autoplaced)
+    (effects (font (size 1.27 1.27)) (justify right bottom))
+  )
+  (label "PIO19" (at 151.13 117.475 180) (fields_autoplaced)
+    (effects (font (size 1.27 1.27)) (justify right bottom))
+  )
+  (label "PIO18" (at 151.13 112.395 180) (fields_autoplaced)
+    (effects (font (size 1.27 1.27)) (justify right bottom))
+  )
+  (label "PIO22" (at 151.13 89.535 180) (fields_autoplaced)
+    (effects (font (size 1.27 1.27)) (justify right bottom))
+  )

Commit message: schematic updated
Parts:
- IC1: footprint BGA225C80P15X15_1300X1300X140 -> SamacSys_Parts:BGA225C80P15X15_1300X1300X140
- R20: footprint (none) -> Resistor_SMD:R_0402_1005Metric_Pad0.72x0.64mm_HandSolder
Changed lines of the file:
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@@
       (effects (font (size 1.27 1.27)))
     )
-    (property "Footprint" "BGA225C80P15X15_1300X1300X140" (at 212.09 73.66 0)
+    (property "Footprint" "SamacSys_Parts:BGA225C80P15X15_1300X1300X140" (at 212.09 73.66 0)
       (effects (font (size 1.27 1.27)) (justify left top) hide)
     )
@@
       (effects (font (size 1.27 1.27)))
     )
-    (property "Footprint" "" (at 147.955 81.915 0)
+    (property "Footprint" "Resistor_SMD:R_0402_1005Metric_Pad0.72x0.64mm_HandSolder" (at 147.955 81.915 0)
       (effects (font (size 1.27 1.27)) hide)
     )

Commit message: updated schematic
Connections:
- net UART_RXD_OUT renamed RXD_OUT
- net UART_TXD_IN renamed TXD_IN
Changed lines of the file:
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@@
     (effects (font (size 1.27 1.27)) (justify right bottom))
   )
-  (label "GCLK" (at 145.415 81.915 180) (fields_autoplaced)
+  (label "GCLK" (at 143.51 81.915 180) (fields_autoplaced)
     (effects (font (size 1.27 1.27)) (justify right bottom))
   )
@@
     (effects (font (size 1.27 1.27)) (justify right bottom))
   )
+  (hierarchical_label "TXD_IN" (shape input) (at 151.13 61.595 0) (fields_autoplaced)
+    (effects (font (size 1.27 1.27)) (justify left))
+  )
+  (hierarchical_label "RXD_OUT" (shape input) (at 151.13 66.675 0) (fields_autoplaced)
+    (effects (font (size 1.27 1.27)) (justify left))
+  )
   (symbol (lib_id "SamacSys_Parts:XC7S25-1CSGA225C") (at 103.505 100.965 0) (unit 2)

Commit message: pcb layout updated
Changed lines of the file:
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@@
     (effects (font (size 1.27 1.27)) (justify right bottom))
   )
+  (hierarchical_label "PIO30" (shape input) (at 151.13 86.995 0) (fields_autoplaced)
+    (effects (font (size 1.27 1.27)) (justify left))
+  )
+  (hierarchical_label "PIO22" (shape input) (at 151.13 89.535 0) (fields_autoplaced)
+    (effects (font (size 1.27 1.27)) (justify left))
+  )
+  (hierarchical_label "PIO16" (shape input) (at 151.13 132.715 0) (fields_autoplaced)
+    (effects (font (size 1.27 1.27)) (justify left))
+  )
+  (hierarchical_label "PIO18" (shape input) (at 151.13 112.395 0) (fields_autoplaced)
+    (effects (font (size 1.27 1.27)) (justify left))
+  )
+  (hierarchical_label "PIO23" (shape input) (at 151.13 74.295 0) (fields_autoplaced)
+    (effects (font (size 1.27 1.27)) (justify left))
+  )
   (hierarchical_label "TXD_IN" (shape input) (at 151.13 61.595 0) (fields_autoplaced)
+    (effects (font (size 1.27 1.27)) (justify left))
+  )
+  (hierarchical_label "PIO19" (shape input) (at 151.13 117.475 0) (fields_autoplaced)
+    (effects (font (size 1.27 1.27)) (justify left))
+  )
+  (hierarchical_label "PIO31" (shape input) (at 151.13 53.975 0) (fields_autoplaced)
+    (effects (font (size 1.27 1.27)) (justify left))
+  )
+  (hierarchical_label "PIO27" (shape input) (at 151.13 59.055 0) (fields_autoplaced)
+    (effects (font (size 1.27 1.27)) (justify left))
+  )
+  (hierarchical_label "PIO21" (shape input) (at 151.13 92.075 0) (fields_autoplaced)
+    (effects (font (size 1.27 1.27)) (justify left))
+  )
+  (hierarchical_label "PIO20" (shape input) (at 151.13 114.935 0) (fields_autoplaced)
+    (effects (font (size 1.27 1.27)) (justify left))
+  )
+  (hierarchical_label "PIO29" (shape input) (at 151.13 69.215 0) (fields_autoplaced)
+    (effects (font (size 1.27 1.27)) (justify left))
+  )
+  (hierarchical_label "PIO17" (shape input) (at 151.13 135.255 0) (fields_autoplaced)
+    (effects (font (size 1.27 1.27)) (justify left))
+  )
+  (hierarchical_label "PIO28" (shape input) (at 151.13 56.515 0) (fields_autoplaced)
     (effects (font (size 1.27 1.27)) (justify left))
   )
@@
     (effects (font (size 1.27 1.27)) (justify left))
   )
+  (hierarchical_label "PIO26" (shape input) (at 151.13 71.755 0) (fields_autoplaced)
+    (effects (font (size 1.27 1.27)) (justify left))
+  )
