File: kicad_files/BANK_15.kicad_sch (KiCad schematic)
At the start: 1 part, among them IC1 XC7S25-1CSGA225C

Commit message: schematic updated
Changed lines of the file:
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@@
   (symbol (lib_id "SamacSys_Parts:XC7S25-1CSGA225C") (at 105.41 109.855 0) (unit 3)
     (in_bom yes) (on_board yes) (dnp no)
-    (property "Reference" "IC1" (at 105.41 33.02 0)
+    (property "Reference" "IC1" (at 102.87 52.07 0)
       (effects (font (size 1.27 1.27)))
     )
-    (property "Value" "XC7S25-1CSGA225C" (at 105.41 36.195 0)
+    (property "Value" "XC7S25-1CSGA225C" (at 102.87 55.245 0)
       (effects (font (size 1.27 1.27)))
     )
@@
     (pin "R1")
     (pin "R15")
-    (pin "E5")
-    (pin "F5")
-    (pin "G5")
-    (pin "G8")
-    (pin "G9")
-    (pin "H14")
-    (pin "H15")
-    (pin "H5")
-    (pin "H8")
-    (pin "H9")
     (pin "J11")
-    (pin "J12")
     (pin "J15")
-    (pin "J5")
-    (pin "J8")
-    (pin "J9")
-    (pin "K11")
-    (pin "K12")
-    (pin "K13")
     (pin "K14")
     (pin "K15")
-    (pin "K4")
-    (pin "K5")
     (pin "L10")
-    (pin "L11")
     (pin "L12")
     (pin "L13")
     (pin "L14")
     (pin "L15")
-    (pin "L4")
-    (pin "L5")
     (pin "M10")
     (pin "M13")
     (pin "M14")
     (pin "M15")
-    (pin "M5")
-    (pin "M6")
     (pin "M7")
     (pin "M8")
     (pin "M9")
-    (pin "N10")
-    (pin "N11")
     (pin "N12")
     (pin "N13")
     (pin "N14")
     (pin "N15")
-    (pin "N5")
     (pin "N6")
     (pin "N7")
     (pin "N8")
     (pin "N9")
-    (pin "P10")
     (pin "P11")
     (pin "P12")
@@
           (reference "IC1") (unit 3)
         )
+        (path "/94bd3a84-5526-4cf2-a5cc-3887356f447c/30d52c37-ae5c-405e-8a78-89b18a6efc4e/af489dd5-0e9e-4b3e-a401-f1288bd8b210"
+          (reference "IC1") (unit 3)
+        )

Commit message: schematic updated
Parts:
- IC1: footprint BGA225C80P15X15_1300X1300X140 -> SamacSys_Parts:BGA225C80P15X15_1300X1300X140
Changed lines of the file:
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@@
       (effects (font (size 1.27 1.27)))
     )
-    (property "Footprint" "BGA225C80P15X15_1300X1300X140" (at 213.995 82.55 0)
+    (property "Footprint" "SamacSys_Parts:BGA225C80P15X15_1300X1300X140" (at 213.995 82.55 0)
       (effects (font (size 1.27 1.27)) (justify left top) hide)
     )

Commit message: updated schematic
Parts:
- added C72, C73: 1uf, symbol Device:C_Small
- added R14 (x2): 1K, Resistor_SMD:R_0402_1005Metric_Pad0.72x0.64mm_HandSolder, symbol Device:R_Small_US
- added R14 (x2): 2.32K, Resistor_SMD:R_0402_1005Metric_Pad0.72x0.64mm_HandSolder, symbol Device:R_Small_US
- added R14 (x2): 140, Resistor_SMD:R_0402_1005Metric_Pad0.72x0.64mm_HandSolder, symbol Device:R_Small_US
- added R14 (x2): 845, Resistor_SMD:R_0402_1005Metric_Pad0.72x0.64mm_HandSolder, symbol Device:R_Small_US
Connections:
- net AIN33_P: now reaches IC1.A11 (IO_L11P_T1_SRCC_AD12P_15)
- net AIN33_P: now also C72.1, R14.2
- net AIN33_N: now reaches IC1.A12 (IO_L11N_T1_SRCC_AD12N_15)
- net AIN33_N: now also C72.2, R14.2
- net AIN32_P: now reaches IC1.A13 (IO_L12P_T1_MRCC_AD5P_15)
- net AIN32_P: now also C73.1, R14.2
- net AIN32_N: now reaches IC1.A14 (IO_L12N_T1_MRCC_AD5N_15)
- net AIN32_N: now also C73.2, R14.2
- new net: R14.1, R14.1, R14.2 (x2)
- new net AIN32: R14.1
- new net AIN33: R14.1
- new net GND: R14.1, R14.1, R14.2, R14.2
- no-connect marks 0 -> 46

Commit message: pcb layout updated
Parts:
- C72, C73: footprint (none) -> Capacitor_SMD:C_0402_1005Metric_Pad0.74x0.62mm_HandSolder
Changed lines of the file:
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@@
       (effects (font (size 1.27 1.27)) (justify left))
     )
-    (property "Footprint" "" (at 196.85 63.5 0)
+    (property "Footprint" "Capacitor_SMD:C_0402_1005Metric_Pad0.74x0.62mm_HandSolder" (at 196.85 63.5 0)
       (effects (font (size 1.27 1.27)) hide)
     )
@@
       (effects (font (size 1.27 1.27)) (justify left))
     )
-    (property "Footprint" "" (at 196.85 82.55 0)
+    (property "Footprint" "Capacitor_SMD:C_0402_1005Metric_Pad0.74x0.62mm_HandSolder" (at 196.85 82.55 0)
       (effects (font (size 1.27 1.27)) hide)
     )
