File: kicad_files/BANK_34.kicad_sch (KiCad schematic)
At the start: 1 part, among them IC2 XC7S25-1CSGA225C

Commit message: schematic updated
Changed lines of the file:
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@@
   (symbol (lib_id "SamacSys_Parts:XC7S25-1CSGA225C") (at 71.12 95.25 0) (unit 4)
     (in_bom yes) (on_board yes) (dnp no)
-    (property "Reference" "IC2" (at 71.12 18.415 0)
+    (property "Reference" "IC2" (at 68.58 37.465 0)
       (effects (font (size 1.27 1.27)))
     )
-    (property "Value" "XC7S25-1CSGA225C" (at 71.12 21.59 0)
+    (property "Value" "XC7S25-1CSGA225C" (at 68.58 40.64 0)
       (effects (font (size 1.27 1.27)))
     )
@@
     (pin "R1")
     (pin "R15")
-    (pin "E5")
-    (pin "F5")
-    (pin "G5")
-    (pin "G8")
-    (pin "G9")
-    (pin "H14")
-    (pin "H15")
-    (pin "H5")
-    (pin "H8")
-    (pin "H9")
     (pin "J11")
-    (pin "J12")
     (pin "J15")
-    (pin "J5")
-    (pin "J8")
-    (pin "J9")
-    (pin "K11")
-    (pin "K12")
-    (pin "K13")
     (pin "K14")
     (pin "K15")
-    (pin "K4")
-    (pin "K5")
     (pin "L10")
-    (pin "L11")
     (pin "L12")
     (pin "L13")
     (pin "L14")
     (pin "L15")
-    (pin "L4")
-    (pin "L5")
     (pin "M10")
     (pin "M13")
     (pin "M14")
     (pin "M15")
-    (pin "M5")
-    (pin "M6")
     (pin "M7")
     (pin "M8")
     (pin "M9")
-    (pin "N10")
-    (pin "N11")
     (pin "N12")
     (pin "N13")
     (pin "N14")
     (pin "N15")
-    (pin "N5")
     (pin "N6")
     (pin "N7")
     (pin "N8")
     (pin "N9")
-    (pin "P10")
     (pin "P11")
     (pin "P12")
@@
           (reference "IC1") (unit 4)
         )
+        (path "/94bd3a84-5526-4cf2-a5cc-3887356f447c/30d52c37-ae5c-405e-8a78-89b18a6efc4e/af489dd5-0e9e-4b3e-a401-f1288bd8b210"
+          (reference "IC1") (unit 4)
+        )

Commit message: schematic updated
Parts:
- IC2: footprint BGA225C80P15X15_1300X1300X140 -> SamacSys_Parts:BGA225C80P15X15_1300X1300X140
Changed lines of the file:
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@@
       (effects (font (size 1.27 1.27)))
     )
-    (property "Footprint" "BGA225C80P15X15_1300X1300X140" (at 179.705 67.945 0)
+    (property "Footprint" "SamacSys_Parts:BGA225C80P15X15_1300X1300X140" (at 179.705 67.945 0)
       (effects (font (size 1.27 1.27)) (justify left top) hide)
     )

Commit message: updated schematic
Connections:
- net PIO41: now reaches IC2.A2 (IO_L2N_T0_34)
- net PIO47: now reaches IC2.A3 (IO_L1N_T0_34)
- net PIO48: now reaches IC2.A4 (IO_L1P_T0_34)
- net PIO43: now reaches IC2.B1 (IO_L4N_T0_34)
- net PIO42: now reaches IC2.B2 (IO_L2P_T0_34)
- net PIO45: now reaches IC2.B3 (IO_L3N_T0_DQS_34)
- net PIO46: now reaches IC2.B4 (IO_L3P_T0_DQS_34)
- net PIO44: now reaches IC2.C1 (IO_L4P_T0_34)
- net PIO40: now reaches IC2.C5 (IO_L5P_T0_34)
- net BTN1: now reaches IC2.D1 (IO_L6N_T0_VREF_34)
- net BTN0: now reaches IC2.D2 (IO_L6P_T0_34)
- net LED0_G: now reaches IC2.D3 (IO_L9N_T1_DQS_34)
- net LED4: now reaches IC2.E1 (IO_L8N_T1_34)
- net LED1: now reaches IC2.E2 (IO_L8P_T1_34)
- net LED1: now also IC2.K1 (IO_L16P_T2_34)
- net LED0_B: now reaches IC2.F1 (IO_L10N_T1_34)
- net LED0_R: now reaches IC2.F2 (IO_L10P_T1_34)
- net JA4: now reaches IC2.F3 (IO_L11N_T1_SRCC_34)
- net JA10: now reaches IC2.F4 (IO_L11P_T1_SRCC_34)
- net JA9: now reaches IC2.G1 (IO_L12N_T1_MRCC_34)
- net JA8: now reaches IC2.H1 (IO_L12P_T1_MRCC_34)
- net JA2: now reaches IC2.H2 (IO_L14N_T2_SRCC_34)
- net JA7: now reaches IC2.H3 (IO_L13N_T2_MRCC_34)
- net JA3: now reaches IC2.H4 (IO_L13P_T2_MRCC_34)
- net LED3: now reaches IC2.J1 (IO_L16N_T2_34)
- net JA1: now reaches IC2.J2 (IO_L14P_T2_SRCC_34)
- net PIO01: now reaches IC2.L1 (IO_L18N_T2_34)
- net PIO05: now reaches IC2.M2 (IO_L20N_T3_34)
- net PIO03: now reaches IC2.M3 (IO_L19N_T3_VREF_34)
- net PIO02: now reaches IC2.M4 (IO_L19P_T3_34)
- net PIO09: now reaches IC2.N1 (IO_L22N_T3_34)
- net PIO04: now reaches IC2.N2 (IO_L20P_T3_34)
- net PIO07: now reaches IC2.N3 (IO_L21N_T3_DQS_34)
- net PIO08: now reaches IC2.P1 (IO_L22P_T3_34)
- net PIO06: now reaches IC2.P3 (IO_L21P_T3_DQS_34)
- no-connect marks 0 -> 15
Changed lines of the file:
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@@
 (kicad_sch (version 20230121) (generator eeschema)
   (paper "A4")
+  (no_connect (at 100.965 86.995))
+  (no_connect (at 100.965 158.115))
+  (no_connect (at 100.965 64.135))
+  (no_connect (at 100.965 71.755))
+  (no_connect (at 100.965 66.675))
+  (no_connect (at 100.965 79.375))
+  (no_connect (at 100.965 122.555))
+  (no_connect (at 100.965 153.035))
+  (no_connect (at 100.965 104.775))
+  (no_connect (at 100.965 163.195))
+  (no_connect (at 100.965 137.795))
+  (no_connect (at 100.965 56.515))
+  (no_connect (at 100.965 74.295))
+  (no_connect (at 100.965 114.935))
+  (no_connect (at 100.965 155.575))
+  (wire (pts (xy 100.965 84.455) (xy 121.285 84.455))
+    (stroke (width 0) (type default))
+  )
+  (wire (pts (xy 100.965 94.615) (xy 121.285 94.615))
+    (stroke (width 0) (type default))
+  )
+  (wire (pts (xy 100.965 135.255) (xy 120.65 135.255))
+    (stroke (width 0) (type default))
+  )
+  (wire (pts (xy 100.965 142.875) (xy 120.65 142.875))
+    (stroke (width 0) (type default))
+  )
+  (wire (pts (xy 100.965 97.155) (xy 121.285 97.155))
+    (stroke (width 0) (type default))
+  )
+  (wire (pts (xy 100.965 69.215) (xy 121.285 69.215))
+    (stroke (width 0) (type default))
+  )
+  (wire (pts (xy 100.965 41.275) (xy 121.285 41.275))
+    (stroke (width 0) (type default))
+  )
+  (wire (pts (xy 100.965 145.415) (xy 120.65 145.415))
+    (stroke (width 0) (type default))
+  )
+  (wire (pts (xy 100.965 76.835) (xy 121.285 76.835))
+    (stroke (width 0) (type default))
+  )
+  (wire (pts (xy 100.965 109.855) (xy 120.65 109.855))
+    (stroke (width 0) (type default))
+  )
+  (wire (pts (xy 100.965 53.975) (xy 121.285 53.975))
+    (stroke (width 0) (type default))
+  )
+  (wire (pts (xy 100.965 81.915) (xy 121.285 81.915))
+    (stroke (width 0) (type default))
+  )
+  (wire (pts (xy 100.965 120.015) (xy 120.65 120.015))
+    (stroke (width 0) (type default))
+  )
+  (wire (pts (xy 100.965 61.595) (xy 121.285 61.595))
+    (stroke (width 0) (type default))
+  )
+  (wire (pts (xy 100.965 89.535) (xy 121.285 89.535))
+    (stroke (width 0) (type default))
+  )
+  (wire (pts (xy 100.965 147.955) (xy 120.65 147.955))
+    (stroke (width 0) (type default))
+  )
+  (wire (pts (xy 100.965 38.735) (xy 121.285 38.735))
+    (stroke (width 0) (type default))
+  )
+  (wire (pts (xy 100.965 48.895) (xy 121.285 48.895))
+    (stroke (width 0) (type default))
+  )
+  (wire (pts (xy 100.965 117.475) (xy 120.65 117.475))
+    (stroke (width 0) (type default))
+  )
+  (wire (pts (xy 100.965 46.355) (xy 121.285 46.355))
+    (stroke (width 0) (type default))
+  )
+  (wire (pts (xy 100.965 127.635) (xy 120.65 127.635))
+    (stroke (width 0) (type default))
+  )
+  (wire (pts (xy 100.965 92.075) (xy 121.285 92.075))
+    (stroke (width 0) (type default))
+  )
+  (wire (pts (xy 100.965 132.715) (xy 120.65 132.715))
+    (stroke (width 0) (type default))
+  )
+  (wire (pts (xy 100.965 107.315) (xy 120.65 107.315))
+    (stroke (width 0) (type default))
+  )
+  (wire (pts (xy 100.965 130.175) (xy 120.65 130.175))
+    (stroke (width 0) (type default))
+  )
+  (wire (pts (xy 100.965 150.495) (xy 120.65 150.495))
+    (stroke (width 0) (type default))
+  )
+  (wire (pts (xy 100.965 59.055) (xy 121.285 59.055))
+    (stroke (width 0) (type default))
+  )
+  (wire (pts (xy 100.965 99.695) (xy 121.285 99.695))
+    (stroke (width 0) (type default))
+  )
+  (wire (pts (xy 100.965 160.655) (xy 120.65 160.655))
+    (stroke (width 0) (type default))
+  )
+  (wire (pts (xy 100.965 51.435) (xy 121.285 51.435))
+    (stroke (width 0) (type default))
+  )
+  (wire (pts (xy 100.965 43.815) (xy 121.285 43.815))
+    (stroke (width 0) (type default))
+  )
+  (wire (pts (xy 100.965 125.095) (xy 120.65 125.095))
+    (stroke (width 0) (type default))
+  )
+  (wire (pts (xy 100.965 140.335) (xy 120.65 140.335))
+    (stroke (width 0) (type default))
+  )
+  (wire (pts (xy 100.965 102.235) (xy 121.285 102.235))
+    (stroke (width 0) (type default))
+  )
+  (wire (pts (xy 100.965 112.395) (xy 120.65 112.395))
+    (stroke (width 0) (type default))
+  )
+  (label "PIO07" (at 120.65 112.395 180) (fields_autoplaced)
+    (effects (font (size 1.27 1.27)) (justify right bottom))
+  )
+  (label "JA1" (at 121.285 61.595 180) (fields_autoplaced)
+    (effects (font (size 1.27 1.27)) (justify right bottom))
+  )
+  (label "PIO01" (at 121.285 84.455 180) (fields_autoplaced)
+    (effects (font (size 1.27 1.27)) (justify right bottom))
+  )
+  (label "BTN1" (at 121.285 97.155 180) (fields_autoplaced)
+    (effects (font (size 1.27 1.27)) (justify right bottom))
+  )
+  (label "LED1" (at 121.285 69.215 180) (fields_autoplaced)
+    (effects (font (size 1.27 1.27)) (justify right bottom))
+  )
+  (label "PIO45" (at 121.285 51.435 180) (fields_autoplaced)
+    (effects (font (size 1.27 1.27)) (justify right bottom))
+  )
+  (label "JA10" (at 120.65 132.715 180) (fields_autoplaced)
+    (effects (font (size 1.27 1.27)) (justify right bottom))
+  )
+  (label "PIO02" (at 121.285 94.615 180) (fields_autoplaced)
+    (effects (font (size 1.27 1.27)) (justify right bottom))
+  )
+  (label "LED3" (at 121.285 59.055 180) (fields_autoplaced)
+    (effects (font (size 1.27 1.27)) (justify right bottom))
+  )
+  (label "JA9" (at 120.65 160.655 180) (fields_autoplaced)
+    (effects (font (size 1.27 1.27)) (justify right bottom))
+  )
+  (label "JA7" (at 120.65 147.955 180) (fields_autoplaced)
+    (effects (font (size 1.27 1.27)) (justify right bottom))
+  )
+  (label "LED0_B" (at 120.65 125.095 180) (fields_autoplaced)
+    (effects (font (size 1.27 1.27)) (justify right bottom))
+  )
+  (label "LED0_R" (at 120.65 127.635 180) (fields_autoplaced)
+    (effects (font (size 1.27 1.27)) (justify right bottom))
+  )
+  (label "PIO09" (at 120.65 107.315 180) (fields_autoplaced)
+    (effects (font (size 1.27 1.27)) (justify right bottom))
+  )
+  (label "PIO43" (at 121.285 46.355 180) (fields_autoplaced)
+    (effects (font (size 1.27 1.27)) (justify right bottom))
+  )
+  (label "PIO48" (at 121.285 43.815 180) (fields_autoplaced)
+    (effects (font (size 1.27 1.27)) (justify right bottom))
+  )
+  (label "PIO08" (at 120.65 135.255 180) (fields_autoplaced)
+    (effects (font (size 1.27 1.27)) (justify right bottom))
+  )
+  (label "PIO06" (at 120.65 140.335 180) (fields_autoplaced)
+    (effects (font (size 1.27 1.27)) (justify right bottom))
+  )
+  (label "PIO40" (at 121.285 81.915 180) (fields_autoplaced)
+    (effects (font (size 1.27 1.27)) (justify right bottom))
+  )
+  (label "LED1" (at 120.65 120.015 180) (fields_autoplaced)
+    (effects (font (size 1.27 1.27)) (justify right bottom))
+  )
+  (label "JA8" (at 120.65 142.875 180) (fields_autoplaced)
+    (effects (font (size 1.27 1.27)) (justify right bottom))
+  )
+  (label "PIO46" (at 121.285 53.975 180) (fields_autoplaced)
+    (effects (font (size 1.27 1.27)) (justify right bottom))
+  )
+  (label "BTN0" (at 121.285 99.695 180) (fields_autoplaced)
+    (effects (font (size 1.27 1.27)) (justify right bottom))
+  )
+  (label "PIO04" (at 120.65 109.855 180) (fields_autoplaced)
+    (effects (font (size 1.27 1.27)) (justify right bottom))
+  )
+  (label "PIO05" (at 121.285 89.535 180) (fields_autoplaced)
+    (effects (font (size 1.27 1.27)) (justify right bottom))
+  )
+  (label "PIO03" (at 121.285 92.075 180) (fields_autoplaced)
+    (effects (font (size 1.27 1.27)) (justify right bottom))
+  )
+  (label "PIO41" (at 121.285 38.735 180) (fields_autoplaced)
+    (effects (font (size 1.27 1.27)) (justify right bottom))
+  )
+  (label "PIO42" (at 121.285 48.895 180) (fields_autoplaced)
+    (effects (font (size 1.27 1.27)) (justify right bottom))
+  )
+  (label "LED0_G" (at 121.285 102.235 180) (fields_autoplaced)
+    (effects (font (size 1.27 1.27)) (justify right bottom))
+  )
+  (label "LED4" (at 120.65 117.475 180) (fields_autoplaced)
+    (effects (font (size 1.27 1.27)) (justify right bottom))
+  )
+  (label "JA3" (at 120.65 150.495 180) (fields_autoplaced)
+    (effects (font (size 1.27 1.27)) (justify right bottom))
+  )
+  (label "PIO47" (at 121.285 41.275 180) (fields_autoplaced)
+    (effects (font (size 1.27 1.27)) (justify right bottom))
+  )
+  (label "JA2" (at 120.65 145.415 180) (fields_autoplaced)
+    (effects (font (size 1.27 1.27)) (justify right bottom))
+  )
+  (label "PIO44" (at 121.285 76.835 180) (fields_autoplaced)
+    (effects (font (size 1.27 1.27)) (justify right bottom))
+  )
+  (label "JA4" (at 120.65 130.175 180) (fields_autoplaced)
+    (effects (font (size 1.27 1.27)) (justify right bottom))
+  )
   (symbol (lib_id "SamacSys_Parts:XC7S25-1CSGA225C") (at 71.12 95.25 0) (unit 4)
     (in_bom yes) (on_board yes) (dnp no)
-    (property "Reference" "IC2" (at 68.58 37.465 0)
+    (property "Reference" "IC2" (at 71.12 22.225 0)
       (effects (font (size 1.27 1.27)))
     )
-    (property "Value" "XC7S25-1CSGA225C" (at 68.58 40.64 0)
+    (property "Value" "XC7S25-1CSGA225C" (at 71.12 25.4 0)
       (effects (font (size 1.27 1.27)))
     )

Commit message: BGA Routing started
Parts:
- added D12: LED_2, LED_SMD:LED_0603_1608Metric_Pad1.05x0.95mm_HandSolder, symbol Device:LED_Small
- added D13: LED_3, LED_SMD:LED_0603_1608Metric_Pad1.05x0.95mm_HandSolder, symbol Device:LED_Small
- added D14: LED_4, LED_SMD:LED_0603_1608Metric_Pad1.05x0.95mm_HandSolder, symbol Device:LED_Small
- added D9: LED_1, LED_SMD:LED_0603_1608Metric_Pad1.05x0.95mm_HandSolder, symbol Device:LED_Small
- added R29 (x4): 330, Resistor_SMD:R_0402_1005Metric_Pad0.72x0.64mm_HandSolder, symbol Device:R_Small_US
Connections:
- net LED1: now also R29.1; no longer IC2.K1 (IO_L16P_T2_34)
- net LED3: now also R29.1
- net LED4: now also R29.1
- new net: D13.2 (A), R29.2
- new net: D14.2 (A), R29.2
- new net: D9.2 (A), R29.2
- new net: D12.2 (A), R29.2
- new net GND: D12.1 (K), D13.1 (K), D14.1 (K), D9.1 (K)
- new net LED2: IC2.K1 (IO_L16P_T2_34), R29.1

Commit message: pcb layout updated
Changed lines of the file:
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@@
     (effects (font (size 1.27 1.27)) (justify left bottom))
+  )
+  (hierarchical_label "JA3" (shape input) (at 120.65 150.495 0) (fields_autoplaced)
+    (effects (font (size 1.27 1.27)) (justify left))
+  )
+  (hierarchical_label "PIO02" (shape input) (at 121.285 94.615 0) (fields_autoplaced)
+    (effects (font (size 1.27 1.27)) (justify left))
+  )
+  (hierarchical_label "PIO45" (shape input) (at 121.285 51.435 0) (fields_autoplaced)
+    (effects (font (size 1.27 1.27)) (justify left))
+  )
+  (hierarchical_label "PIO05" (shape input) (at 121.285 89.535 0) (fields_autoplaced)
+    (effects (font (size 1.27 1.27)) (justify left))
+  )
+  (hierarchical_label "PIO07" (shape input) (at 120.65 112.395 0) (fields_autoplaced)
+    (effects (font (size 1.27 1.27)) (justify left))
+  )
+  (hierarchical_label "JA2" (shape input) (at 120.65 145.415 0) (fields_autoplaced)
+    (effects (font (size 1.27 1.27)) (justify left))
+  )
+  (hierarchical_label "PIO47" (shape input) (at 121.285 41.275 0) (fields_autoplaced)
+    (effects (font (size 1.27 1.27)) (justify left))
+  )
+  (hierarchical_label "PIO08" (shape input) (at 120.65 135.255 0) (fields_autoplaced)
+    (effects (font (size 1.27 1.27)) (justify left))
+  )
+  (hierarchical_label "PIO43" (shape input) (at 121.285 46.355 0) (fields_autoplaced)
+    (effects (font (size 1.27 1.27)) (justify left))
+  )
+  (hierarchical_label "JA8" (shape input) (at 120.65 142.875 0) (fields_autoplaced)
+    (effects (font (size 1.27 1.27)) (justify left))
+  )
+  (hierarchical_label "PIO04" (shape input) (at 120.65 109.855 0) (fields_autoplaced)
+    (effects (font (size 1.27 1.27)) (justify left))
+  )
+  (hierarchical_label "JA10" (shape input) (at 120.65 132.715 0) (fields_autoplaced)
+    (effects (font (size 1.27 1.27)) (justify left))
+  )
+  (hierarchical_label "PIO01" (shape input) (at 121.285 84.455 0) (fields_autoplaced)
+    (effects (font (size 1.27 1.27)) (justify left))
+  )
+  (hierarchical_label "PIO42" (shape input) (at 121.285 48.895 0) (fields_autoplaced)
+    (effects (font (size 1.27 1.27)) (justify left))
+  )
+  (hierarchical_label "PIO41" (shape input) (at 121.285 38.735 0) (fields_autoplaced)
+    (effects (font (size 1.27 1.27)) (justify left))
+  )
+  (hierarchical_label "PIO46" (shape input) (at 121.285 53.975 0) (fields_autoplaced)
+    (effects (font (size 1.27 1.27)) (justify left))
+  )
+  (hierarchical_label "PIO03" (shape input) (at 121.285 92.075 0) (fields_autoplaced)
+    (effects (font (size 1.27 1.27)) (justify left))
+  )
+  (hierarchical_label "JA1" (shape input) (at 121.285 61.595 0) (fields_autoplaced)
+    (effects (font (size 1.27 1.27)) (justify left))
+  )
+  (hierarchical_label "PIO06" (shape input) (at 120.65 140.335 0) (fields_autoplaced)
+    (effects (font (size 1.27 1.27)) (justify left))
+  )
+  (hierarchical_label "PIO40" (shape input) (at 121.285 81.915 0) (fields_autoplaced)
+    (effects (font (size 1.27 1.27)) (justify left))
+  )
+  (hierarchical_label "PIO09" (shape input) (at 120.65 107.315 0) (fields_autoplaced)
+    (effects (font (size 1.27 1.27)) (justify left))
+  )
+  (hierarchical_label "JA4" (shape input) (at 120.65 130.175 0) (fields_autoplaced)
+    (effects (font (size 1.27 1.27)) (justify left))
+  )
+  (hierarchical_label "JA7" (shape input) (at 120.65 147.955 0) (fields_autoplaced)
+    (effects (font (size 1.27 1.27)) (justify left))
+  )
+  (hierarchical_label "JA9" (shape input) (at 120.65 160.655 0) (fields_autoplaced)
+    (effects (font (size 1.27 1.27)) (justify left))
+  )
+  (hierarchical_label "PIO44" (shape input) (at 121.285 76.835 0) (fields_autoplaced)
+    (effects (font (size 1.27 1.27)) (justify left))
+  )
+  (hierarchical_label "PIO48" (shape input) (at 121.285 43.815 0) (fields_autoplaced)
+    (effects (font (size 1.27 1.27)) (justify left))
   )
   (symbol (lib_id "Device:R_Small_US") (at 172.085 73.66 90) (unit 1)
