File: kicad_files/POWER.kicad_sch (KiCad schematic)
At the start: 48 parts, among them IC2 XC7S25-1CSGA225C

Commit message: schematic updated
Connections:
- net VCC1V8: now also FB2.2
Changed lines of the file:
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@@
+    (stroke (width 0) (type default))
+  )
+  (wire (pts (xy 188.595 138.43) (xy 202.565 138.43))
     (stroke (width 0) (type default))
   )
@@
   )
   (label "VCC1V0" (at 226.06 113.03 180) (fields_autoplaced)
+    (effects (font (size 1.27 1.27)) (justify right bottom))
+  )
+  (label "VCC1V8" (at 202.565 138.43 180) (fields_autoplaced)
     (effects (font (size 1.27 1.27)) (justify right bottom))
   )
@@
   (symbol (lib_id "SamacSys_Parts:XC7S25-1CSGA225C") (at 120.015 90.17 0) (unit 1)
     (in_bom yes) (on_board yes) (dnp no)
-    (property "Reference" "IC2" (at 120.015 13.335 0)
+    (property "Reference" "IC2" (at 117.475 32.385 0)
       (effects (font (size 1.27 1.27)))
     )
-    (property "Value" "XC7S25-1CSGA225C" (at 120.015 16.51 0)
+    (property "Value" "XC7S25-1CSGA225C" (at 117.475 35.56 0)
       (effects (font (size 1.27 1.27)))
     )
@@
     (pin "R1")
     (pin "R15")
-    (pin "E5")
-    (pin "F5")
-    (pin "G5")
-    (pin "G8")
-    (pin "G9")
-    (pin "H14")
-    (pin "H15")
-    (pin "H5")
-    (pin "H8")
-    (pin "H9")
     (pin "J11")
-    (pin "J12")
     (pin "J15")
-    (pin "J5")
-    (pin "J8")
-    (pin "J9")
-    (pin "K11")
-    (pin "K12")
-    (pin "K13")
     (pin "K14")
     (pin "K15")
-    (pin "K4")
-    (pin "K5")
     (pin "L10")
-    (pin "L11")
     (pin "L12")
     (pin "L13")
     (pin "L14")
     (pin "L15")
-    (pin "L4")
-    (pin "L5")
     (pin "M10")
     (pin "M13")
     (pin "M14")
     (pin "M15")
-    (pin "M5")
-    (pin "M6")
     (pin "M7")
     (pin "M8")
     (pin "M9")
-    (pin "N10")
-    (pin "N11")
     (pin "N12")
     (pin "N13")
     (pin "N14")
     (pin "N15")
-    (pin "N5")
     (pin "N6")
     (pin "N7")
     (pin "N8")
     (pin "N9")
-    (pin "P10")
     (pin "P11")
     (pin "P12")
@@
           (reference "IC1") (unit 1)
         )
+        (path "/94bd3a84-5526-4cf2-a5cc-3887356f447c/30d52c37-ae5c-405e-8a78-89b18a6efc4e/af489dd5-0e9e-4b3e-a401-f1288bd8b210"
+          (reference "IC1") (unit 1)
+        )

Commit message: schematic updated
Parts:
- C10, C11, C12, C13, C14, C15, C16, C17, C18, C19, C20, C21, C22, C23, C24, C25, C26, C27, C28, C29, C30, C31, C32, C33, C34, C35, C36, C37, C38, C39, C40, C41, C42, C43, C7, C8, C9: footprint (none) -> Capacitor_SMD:C_0402_1005Metric_Pad0.74x0.62mm_HandSolder
- IC?: renamed from IC2; footprint BGA225C80P15X15_1300X1300X140 -> SamacSys_Parts:BGA225C80P15X15_1300X1300X140
- R1, R2: footprint (none) -> Resistor_SMD:R_0402_1005Metric_Pad0.72x0.64mm_HandSolder

Commit message: updated schematic
Other:
- note added: "External Nets"
Changed lines of the file:
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@@
+    (stroke (width 0) (type default))
+  )
+  (polyline (pts (xy 15.875 146.05) (xy 80.645 146.05))
     (stroke (width 0) (type default))
   )
@@
     (stroke (width 0) (type default))
   )
-  (wire (pts (xy 254 148.59) (xy 254 155.575))
+  (wire (pts (xy 53.975 162.56) (xy 53.975 169.545))
     (stroke (width 0) (type default))
   )
@@
     (stroke (width 0) (type default))
   )
-  (wire (pts (xy 228.6 148.59) (xy 254 148.59))
+  (wire (pts (xy 28.575 162.56) (xy 53.975 162.56))
     (stroke (width 0) (type default))
   )
@@
     (stroke (width 0) (type default))
   )
+  (polyline (pts (xy 15.875 146.05) (xy 15.875 193.04))
+    (stroke (width 0) (type default))
+  )
   (wire (pts (xy 157.48 113.03) (xy 164.465 113.03))
     (stroke (width 0) (type default))
@@
     (stroke (width 0) (type default))
   )
+  (polyline (pts (xy 80.645 193.04) (xy 15.875 193.04))
+    (stroke (width 0) (type default))
+  )
   (wire (pts (xy 248.285 33.655) (xy 248.285 36.83))
     (stroke (width 0) (type default))
@@
     (stroke (width 0) (type default))
   )
-  (wire (pts (xy 228.6 139.065) (xy 254 139.065))
+  (wire (pts (xy 28.575 153.035) (xy 53.975 153.035))
     (stroke (width 0) (type default))
   )
@@
     (stroke (width 0) (type default))
   )
+  (polyline (pts (xy 80.645 146.05) (xy 80.645 193.04))
+    (stroke (width 0) (type default))
+  )
   (wire (pts (xy 208.28 49.53) (xy 208.28 53.34))
     (stroke (width 0) (type default))
@@
     (stroke (width 0) (type default))
   )
-  (wire (pts (xy 228.6 145.415) (xy 254 145.415))
-    (stroke (width 0) (type default))
-  )
-  (wire (pts (xy 228.6 142.24) (xy 254 142.24))
+  (wire (pts (xy 28.575 159.385) (xy 53.975 159.385))
+    (stroke (width 0) (type default))
+  )
+  (wire (pts (xy 28.575 156.21) (xy 53.975 156.21))
     (stroke (width 0) (type default))
   )
@@
   (wire (pts (xy 157.48 102.235) (xy 147.32 102.235))
     (stroke (width 0) (type default))
+  )
+  (text "External Nets\n" (at 21.59 187.325 0)
+    (effects (font (size 3 3) (thickness 0.6) bold) (justify left bottom))
   )
   (label "VCC1V0" (at 226.06 113.03 180) (fields_autoplaced)
@@
     (effects (font (size 1.27 1.27)) (justify right bottom))
   )
-  (label "GND" (at 228.6 148.59 0) (fields_autoplaced)
+  (label "GND" (at 28.575 162.56 0) (fields_autoplaced)
     (effects (font (size 1.27 1.27)) (justify left bottom))
   )
@@
     (effects (font (size 1.27 1.27)) (justify right bottom))
   )
-  (label "VCC1V8" (at 228.6 142.24 0) (fields_autoplaced)
+  (label "VCC1V8" (at 28.575 156.21 0) (fields_autoplaced)
     (effects (font (size 1.27 1.27)) (justify left bottom))
   )
@@
     (effects (font (size 1.27 1.27)) (justify right bottom))
   )
-  (label "VCC1V0" (at 228.6 139.065 0) (fields_autoplaced)
+  (label "VCC1V0" (at 28.575 153.035 0) (fields_autoplaced)
     (effects (font (size 1.27 1.27)) (justify left bottom))
   )
-  (label "VCC3V3" (at 228.6 145.415 0) (fields_autoplaced)
+  (label "VCC3V3" (at 28.575 159.385 0) (fields_autoplaced)
     (effects (font (size 1.27 1.27)) (justify left bottom))
   )
@@
     (effects (font (size 1.27 1.27)) (justify right bottom))
   )
-  (hierarchical_label "VCC1V0" (shape output) (at 254 139.065 0) (fields_autoplaced)
+  (hierarchical_label "VCC1V0" (shape output) (at 53.975 153.035 0) (fields_autoplaced)
     (effects (font (size 1.27 1.27)) (justify left))
   )
-  (hierarchical_label "VCC1V8" (shape output) (at 254 142.24 0) (fields_autoplaced)
+  (hierarchical_label "VCC1V8" (shape output) (at 53.975 156.21 0) (fields_autoplaced)
     (effects (font (size 1.27 1.27)) (justify left))
   )
-  (hierarchical_label "VCC3V3" (shape output) (at 254 145.415 0) (fields_autoplaced)
+  (hierarchical_label "VCC3V3" (shape output) (at 53.975 159.385 0) (fields_autoplaced)
     (effects (font (size 1.27 1.27)) (justify left))
   )
@@
   (symbol (lib_id "SamacSys_Parts:XC7S25-1CSGA225C") (at 120.015 90.17 0) (unit 1)
     (in_bom yes) (on_board yes) (dnp no)
-    (property "Reference" "IC?" (at 117.475 32.385 0)
+    (property "Reference" "IC?" (at 120.015 17.78 0)
       (effects (font (size 1.27 1.27)))
     )
-    (property "Value" "XC7S25-1CSGA225C" (at 117.475 35.56 0)
+    (property "Value" "XC7S25-1CSGA225C" (at 120.015 20.955 0)
       (effects (font (size 1.27 1.27)))
     )
@@
     )
   )
-  (symbol (lib_id "power:GND") (at 254 155.575 0) (unit 1)
+  (symbol (lib_id "power:GND") (at 53.975 169.545 0) (unit 1)
     (in_bom yes) (on_board yes) (dnp no)
-    (property "Reference" "#PWR020" (at 254 161.925 0)
-      (effects (font (size 1.27 1.27)) hide)
-    )
-    (property "Value" "GND" (at 254 159.385 0)
+    (property "Reference" "#PWR020" (at 53.975 175.895 0)
+      (effects (font (size 1.27 1.27)) hide)
+    )
+    (property "Value" "GND" (at 53.975 173.355 0)
       (effects (font (size 1.27 1.27)))
     )
-    (property "Footprint" "" (at 254 155.575 0)
-      (effects (font (size 1.27 1.27)) hide)
-    )
-    (property "Datasheet" "" (at 254 155.575 0)
-      (effects (font (size 1.27 1.27)) hide)
-    )
+    (property "Footprint" "" (at 53.975 169.545 0)
+      (effects (font (size 1.27 1.27)) hide)
+    )
+    (property "Datasheet" "" (at 53.975 169.545 0)
+      (effects (font (size 1.27 1.27)) hide)
+    )

Commit message: BGA Routing started
Parts:
- FB1: footprint (none) -> LED_SMD:LED_0603_1608Metric_Pad1.05x0.95mm_HandSolder
Changed lines of the file:
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@@
       (effects (font (size 1.27 1.27)))
     )
-    (property "Footprint" "" (at 84.455 138.43 0)
+    (property "Footprint" "LED_SMD:LED_0603_1608Metric_Pad1.05x0.95mm_HandSolder" (at 84.455 138.43 0)
       (effects (font (size 1.27 1.27)) hide)
     )

Commit message: pcb layout updated
Parts:
- C1, C2, C3, C6: footprint (none) -> Capacitor_SMD:C_0402_1005Metric_Pad0.74x0.62mm_HandSolder
- C4: footprint (none) -> Capacitor_SMD:C_0603_1608Metric
- C5: footprint (none) -> Capacitor_SMD:C_1210_3225Metric
- FB1: footprint LED_SMD:LED_0603_1608Metric_Pad1.05x0.95mm_HandSolder -> Inductor_SMD:L_0603_1608Metric_Pad1.05x0.95mm_HandSolder
- FB2: footprint (none) -> Inductor_SMD:L_0603_1608Metric_Pad1.05x0.95mm_HandSolder
Changed lines of the file:
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@@
       (effects (font (size 1.27 1.27)) (justify left))
     )
-    (property "Footprint" "" (at 176.53 121.285 0)
+    (property "Footprint" "Capacitor_SMD:C_0402_1005Metric_Pad0.74x0.62mm_HandSolder" (at 176.53 121.285 0)
       (effects (font (size 1.27 1.27)) hide)
     )
@@
       (effects (font (size 1.27 1.27)) (justify left))
     )
-    (property "Footprint" "" (at 155.575 146.685 0)
+    (property "Footprint" "Capacitor_SMD:C_0402_1005Metric_Pad0.74x0.62mm_HandSolder" (at 155.575 146.685 0)
       (effects (font (size 1.27 1.27)) hide)
     )
@@
       (effects (font (size 1.27 1.27)) (justify left))
     )
-    (property "Footprint" "" (at 200.66 121.285 0)
+    (property "Footprint" "Capacitor_SMD:C_0603_1608Metric" (at 200.66 121.285 0)
       (effects (font (size 1.27 1.27)) hide)
     )
@@
       (effects (font (size 1.27 1.27)) (justify left))
     )
-    (property "Footprint" "" (at 169.545 146.685 0)
+    (property "Footprint" "Capacitor_SMD:C_0402_1005Metric_Pad0.74x0.62mm_HandSolder" (at 169.545 146.685 0)
       (effects (font (size 1.27 1.27)) hide)
     )
@@
       (effects (font (size 1.27 1.27)))
     )
-    (property "Footprint" "" (at 184.785 138.43 0)
+    (property "Footprint" "Inductor_SMD:L_0603_1608Metric_Pad1.05x0.95mm_HandSolder" (at 184.785 138.43 0)
       (effects (font (size 1.27 1.27)) hide)
     )
@@
       (effects (font (size 1.27 1.27)))
     )
-    (property "Footprint" "LED_SMD:LED_0603_1608Metric_Pad1.05x0.95mm_HandSolder" (at 84.455 138.43 0)
+    (property "Footprint" "Inductor_SMD:L_0603_1608Metric_Pad1.05x0.95mm_HandSolder" (at 84.455 138.43 0)
       (effects (font (size 1.27 1.27)) hide)
     )
@@
       (effects (font (size 1.27 1.27)) (justify left))
     )
-    (property "Footprint" "" (at 164.465 121.285 0)
+    (property "Footprint" "Capacitor_SMD:C_0402_1005Metric_Pad0.74x0.62mm_HandSolder" (at 164.465 121.285 0)
       (effects (font (size 1.27 1.27)) hide)
     )
@@
       (effects (font (size 1.27 1.27)) (justify left))
     )
-    (property "Footprint" "" (at 213.36 121.285 0)
-      (effects (font (size 1.27 1.27)) hide)
-    )
+    (property "Footprint" "Capacitor_SMD:C_1210_3225Metric" (at 213.36 121.285 0)
+      (effects (font (size 1.27 1.27)) hide)
+    )

Commit message: updated layout
Parts:
- C10, C11, C18: footprint Capacitor_SMD:C_0402_1005Metric_Pad0.74x0.62mm_HandSolder -> Capacitor_SMD:C_0603_1608Metric_Pad1.08x0.95mm_HandSolder
Changed lines of the file:
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@@
       (effects (font (size 1.27 1.27)) (justify left))
     )
-    (property "Footprint" "Capacitor_SMD:C_0402_1005Metric_Pad0.74x0.62mm_HandSolder" (at 203.835 92.71 0)
+    (property "Footprint" "Capacitor_SMD:C_0603_1608Metric_Pad1.08x0.95mm_HandSolder" (at 203.835 92.71 0)
       (effects (font (size 1.27 1.27)) hide)
     )
@@
       (effects (font (size 1.27 1.27)) (justify left))
     )
-    (property "Footprint" "Capacitor_SMD:C_0402_1005Metric_Pad0.74x0.62mm_HandSolder" (at 203.835 104.775 0)
+    (property "Footprint" "Capacitor_SMD:C_0603_1608Metric_Pad1.08x0.95mm_HandSolder" (at 203.835 104.775 0)
       (effects (font (size 1.27 1.27)) hide)
     )
@@
       (effects (font (size 1.27 1.27)) (justify left))
     )
-    (property "Footprint" "Capacitor_SMD:C_0402_1005Metric_Pad0.74x0.62mm_HandSolder" (at 215.265 104.775 0)
-      (effects (font (size 1.27 1.27)) hide)
-    )
+    (property "Footprint" "Capacitor_SMD:C_0603_1608Metric_Pad1.08x0.95mm_HandSolder" (at 215.265 104.775 0)
+      (effects (font (size 1.27 1.27)) hide)
+    )

Commit message: layout basic completed
Parts:
- C27, C28, C42, C43, C7: footprint Capacitor_SMD:C_0402_1005Metric_Pad0.74x0.62mm_HandSolder -> Capacitor_SMD:C_0603_1608Metric_Pad1.08x0.95mm_HandSolder
- C29: footprint Capacitor_SMD:C_0402_1005Metric_Pad0.74x0.62mm_HandSolder -> Capacitor_SMD:C_1206_3216Metric_Pad1.33x1.80mm_HandSolder
- C4: footprint Capacitor_SMD:C_0603_1608Metric -> Capacitor_SMD:C_0603_1608Metric_Pad1.08x0.95mm_HandSolder
- C5: footprint Capacitor_SMD:C_1210_3225Metric -> Capacitor_SMD:C_1206_3216Metric_Pad1.33x1.80mm_HandSolder
Changed lines of the file:
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@@
       (effects (font (size 1.27 1.27)) (justify left))
     )
-    (property "Footprint" "Capacitor_SMD:C_0402_1005Metric_Pad0.74x0.62mm_HandSolder" (at 238.125 39.37 0)
+    (property "Footprint" "Capacitor_SMD:C_0603_1608Metric_Pad1.08x0.95mm_HandSolder" (at 238.125 39.37 0)
       (effects (font (size 1.27 1.27)) hide)
     )
@@
       (effects (font (size 1.27 1.27)) (justify left))
     )
-    (property "Footprint" "Capacitor_SMD:C_0603_1608Metric" (at 200.66 121.285 0)
+    (property "Footprint" "Capacitor_SMD:C_0603_1608Metric_Pad1.08x0.95mm_HandSolder" (at 200.66 121.285 0)
       (effects (font (size 1.27 1.27)) hide)
     )
@@
       (effects (font (size 1.27 1.27)) (justify left))
     )
-    (property "Footprint" "Capacitor_SMD:C_0402_1005Metric_Pad0.74x0.62mm_HandSolder" (at 190.5 121.285 0)
+    (property "Footprint" "Capacitor_SMD:C_0603_1608Metric_Pad1.08x0.95mm_HandSolder" (at 190.5 121.285 0)
       (effects (font (size 1.27 1.27)) hide)
     )
@@
       (effects (font (size 1.27 1.27)) (justify left))
     )
-    (property "Footprint" "Capacitor_SMD:C_0402_1005Metric_Pad0.74x0.62mm_HandSolder" (at 238.125 72.39 0)
+    (property "Footprint" "Capacitor_SMD:C_0603_1608Metric_Pad1.08x0.95mm_HandSolder" (at 238.125 72.39 0)
       (effects (font (size 1.27 1.27)) hide)
     )
@@
       (effects (font (size 1.27 1.27)) (justify left))
     )
-    (property "Footprint" "Capacitor_SMD:C_0402_1005Metric_Pad0.74x0.62mm_HandSolder" (at 228.6 72.39 0)
+    (property "Footprint" "Capacitor_SMD:C_0603_1608Metric_Pad1.08x0.95mm_HandSolder" (at 228.6 72.39 0)
       (effects (font (size 1.27 1.27)) hide)
     )
@@
       (effects (font (size 1.27 1.27)) (justify left))
     )
-    (property "Footprint" "Capacitor_SMD:C_0402_1005Metric_Pad0.74x0.62mm_HandSolder" (at 228.6 39.37 0)
+    (property "Footprint" "Capacitor_SMD:C_0603_1608Metric_Pad1.08x0.95mm_HandSolder" (at 228.6 39.37 0)
       (effects (font (size 1.27 1.27)) hide)
     )
@@
       (effects (font (size 1.27 1.27)) (justify left))
     )
-    (property "Footprint" "Capacitor_SMD:C_0402_1005Metric_Pad0.74x0.62mm_HandSolder" (at 248.285 39.37 0)
+    (property "Footprint" "Capacitor_SMD:C_1206_3216Metric_Pad1.33x1.80mm_HandSolder" (at 248.285 39.37 0)
       (effects (font (size 1.27 1.27)) hide)
     )
@@
       (effects (font (size 1.27 1.27)) (justify left))
     )
-    (property "Footprint" "Capacitor_SMD:C_1210_3225Metric" (at 213.36 121.285 0)
-      (effects (font (size 1.27 1.27)) hide)
-    )
+    (property "Footprint" "Capacitor_SMD:C_1206_3216Metric_Pad1.33x1.80mm_HandSolder" (at 213.36 121.285 0)
+      (effects (font (size 1.27 1.27)) hide)
+    )
