File: kicad_files/sparton_7.kicad_pcb (KiCad board)
At the start: 2 copper layers, 1 part, among them IC1 XC7S100-1FGGA484C_mod

Commit message: working
Parts:
- IC1: value XC7S100-1FGGA484C_mod -> XC7S25-1CSGA225C; footprint SamacSys_Parts:BGA484C100P22X22_2300X2300X260 -> SamacSys_Parts:BGA225C80P15X15_1300X1300X140
- moved IC1 25.9 mm to (145.3, 80.0)
Routing:
- net unconnected-(IC1-IO_L12P_T1_MRCC_34-PadH1): track 0.66 -> 0.00 mm, vias 1 -> 0

Commit message: ftdi progess
Parts:
- added IC2: FT2232H-56Q-TRAY, SamacSys_Parts:QFN50P800X800X100-57N-D, F.Cu at (136.1, 56.2)
- added U1: MX25L3233FM2I-08G, footprints:SOP8L_200MIL_6110-1406_MAC, F.Cu at (123.8, 54.5)
- moved IC1 43.3 mm to (126.5, 41.0)
Connections:
- IC1 pad A1: unconnected-(IC1-GND_1-PadA1) -> /FPGA_SPARTAN_7/POWER/GND
- IC1 pad A15: unconnected-(IC1-GND_2-PadA15) -> /FPGA_SPARTAN_7/POWER/GND
- IC1 pad B7: unconnected-(IC1-VCCO_15_1-PadB7) -> Net-(IC1A-VCCO_15_1)
- IC1 pad B8: unconnected-(IC1-GND_3-PadB8) -> /FPGA_SPARTAN_7/POWER/GND
- IC1 pad C11: unconnected-(IC1-VCCO_15_2-PadC11) -> Net-(IC1A-VCCO_15_1)
- IC1 pad C12: unconnected-(IC1-GND_5-PadC12) -> /FPGA_SPARTAN_7/POWER/GND
- IC1 pad C2: unconnected-(IC1-GND_4-PadC2) -> /FPGA_SPARTAN_7/POWER/GND
- IC1 pad C3: unconnected-(IC1-VCCO_34_1-PadC3) -> /FPGA_SPARTAN_7/POWER/VCC3V3
- IC1 pad D14: unconnected-(IC1-GND_7-PadD14) -> /FPGA_SPARTAN_7/POWER/GND
- IC1 pad D5: unconnected-(IC1-VCCBATT_0-PadD5) -> Net-(IC1A-VCCBATT_0)
- IC1 pad D6: unconnected-(IC1-GND_6-PadD6) -> /FPGA_SPARTAN_7/POWER/GND
- IC1 pad E10: unconnected-(IC1-VCCINT_2-PadE10) -> /FPGA_SPARTAN_7/POWER/VCC1V0
- IC1 pad E4: unconnected-(IC1-GND_8-PadE4) -> /FPGA_SPARTAN_7/POWER/GND
- IC1 pad E5: unconnected-(IC1-TCK_0-PadE5) -> /FPGA_SPARTAN_7/CONFIG/TCLK
- IC1 pad E6: unconnected-(IC1-VCCO_0_1-PadE6) -> /FPGA_SPARTAN_7/POWER/VCC3V3
- IC1 pad E7: unconnected-(IC1-GND_9-PadE7) -> /FPGA_SPARTAN_7/POWER/GND
- IC1 pad E8: unconnected-(IC1-VCCINT_1-PadE8) -> /FPGA_SPARTAN_7/POWER/VCC1V0
- IC1 pad E9: unconnected-(IC1-GND_10-PadE9) -> /FPGA_SPARTAN_7/POWER/GND
- IC1 pad F10: unconnected-(IC1-GND_12-PadF10) -> /FPGA_SPARTAN_7/POWER/GND
- IC1 pad F12: unconnected-(IC1-VCCO_15_3-PadF12) -> Net-(IC1A-VCCO_15_1)
- IC1 pad F13: unconnected-(IC1-GND_13-PadF13) -> /FPGA_SPARTAN_7/POWER/GND
- IC1 pad F5: unconnected-(IC1-CCLK_0-PadF5) -> /FPGA_SPARTAN_7/CONFIG/QSPI_SCK
- IC1 pad F6: unconnected-(IC1-GND_11-PadF6) -> /FPGA_SPARTAN_7/POWER/GND
- IC1 pad F7: unconnected-(IC1-VCCINT_3-PadF7) -> /FPGA_SPARTAN_7/POWER/VCC1V0
- IC1 pad F8: unconnected-(IC1-GNDADC_0-PadF8) -> Net-(IC1A-GNDADC_0)
- IC1 pad F9: unconnected-(IC1-VCCADC_0-PadF9) -> Net-(IC1A-VCCADC_0)
- IC1 pad G10: unconnected-(IC1-VCCINT_4-PadG10) -> /FPGA_SPARTAN_7/POWER/VCC1V0
- IC1 pad G2: unconnected-(IC1-VCCO_34_2-PadG2) -> /FPGA_SPARTAN_7/POWER/VCC3V3
- IC1 pad G3: unconnected-(IC1-GND_14-PadG3) -> /FPGA_SPARTAN_7/POWER/GND
- IC1 pad G5: unconnected-(IC1-DONE_0-PadG5) -> /FPGA_SPARTAN_7/CONFIG/DONE
- IC1 pad G6: unconnected-(IC1-VCCBRAM_1-PadG6) -> /FPGA_SPARTAN_7/POWER/VCC1V0
- IC1 pad G7: unconnected-(IC1-GND_15-PadG7) -> /FPGA_SPARTAN_7/POWER/GND
- IC1 pad G8: unconnected-(IC1-VREFN_0-PadG8) -> /FPGA_SPARTAN_7/CONFIG/XADCGND
- IC1 pad G9: unconnected-(IC1-VP_0-PadG9) -> /FPGA_SPARTAN_7/CONFIG/XADCGND
- IC1 pad H10: unconnected-(IC1-GND_17-PadH10) -> /FPGA_SPARTAN_7/POWER/GND
- IC1 pad H14: unconnected-(IC1-IO_L1P_T0_D00_MOSI_14-PadH14) -> /FPGA_SPARTAN_7/CONFIG/QSPI_DQ0
- IC1 pad H15: unconnected-(IC1-IO_L1N_T0_D01_DIN_14-PadH15) -> /FPGA_SPARTAN_7/CONFIG/QSPI_DQ1
- IC1 pad H5: unconnected-(IC1-CFGBVS_0-PadH5) -> Net-(IC1E-CFGBVS_0)
- IC1 pad H6: unconnected-(IC1-GND_16-PadH6) -> /FPGA_SPARTAN_7/POWER/GND
- IC1 pad H7: unconnected-(IC1-VCCINT_5-PadH7) -> /FPGA_SPARTAN_7/POWER/VCC1V0
- IC1 pad H8: unconnected-(IC1-VN_0-PadH8) -> /FPGA_SPARTAN_7/CONFIG/XADCGND
- IC1 pad H9: unconnected-(IC1-VREFP_0-PadH9) -> /FPGA_SPARTAN_7/CONFIG/XADCGND
- IC1 pad J10: unconnected-(IC1-VCCINT_6-PadJ10) -> /FPGA_SPARTAN_7/POWER/VCC1V0
- IC1 pad J11: unconnected-(IC1-IO_0_14-PadJ11) -> /FPGA_SPARTAN_7/BANK_14/PIO31
- IC1 pad J12: unconnected-(IC1-IO_L2P_T0_D02_14-PadJ12) -> /FPGA_SPARTAN_7/CONFIG/QSPI_DQ2
- IC1 pad J13: unconnected-(IC1-GND_19-PadJ13) -> /FPGA_SPARTAN_7/POWER/GND
- IC1 pad J14: unconnected-(IC1-VCCO_14_1-PadJ14) -> /FPGA_SPARTAN_7/POWER/VCC3V3
- IC1 pad J15: unconnected-(IC1-IO_L5P_T0_D06_14-PadJ15) -> /FPGA_SPARTAN_7/BANK_14/PIO28
- IC1 pad J5: unconnected-(IC1-PROGRAM_B_0-PadJ5) -> /FPGA_SPARTAN_7/CONFIG/PROG
- IC1 pad J6: unconnected-(IC1-VCCBRAM_2-PadJ6) -> /FPGA_SPARTAN_7/POWER/VCC1V0
- IC1 pad J7: unconnected-(IC1-GND_18-PadJ7) -> /FPGA_SPARTAN_7/POWER/GND
- IC1 pad J8: unconnected-(IC1-DXN_0-PadJ8) -> /FPGA_SPARTAN_7/CONFIG/GND
- IC1 pad J9: unconnected-(IC1-DXP_0-PadJ9) -> /FPGA_SPARTAN_7/CONFIG/GND
- IC1 pad K10: unconnected-(IC1-GND_22-PadK10) -> /FPGA_SPARTAN_7/POWER/GND
- IC1 pad K11: unconnected-(IC1-IO_L3P_T0_DQS_PUDC_B_14-PadK11) -> Net-(IC1E-IO_L3P_T0_DQS_PUDC_B_14)
- IC1 pad K12: unconnected-(IC1-IO_L3N_T0_DQS_EMCCLK_14-PadK12) -> Net-(IC1E-IO_L3N_T0_DQS_EMCCLK_14)
- IC1 pad K13: unconnected-(IC1-IO_L2N_T0_D03_14-PadK13) -> /FPGA_SPARTAN_7/CONFIG/QSPI_DQ3
- IC1 pad K14: unconnected-(IC1-IO_L4P_T0_D04_14-PadK14) -> /FPGA_SPARTAN_7/BANK_14/PIO27
- IC1 pad K15: unconnected-(IC1-IO_L5N_T0_D07_14-PadK15) -> /FPGA_SPARTAN_7/BANK_14/UART_TXD_IN
- IC1 pad K4: unconnected-(IC1-TDO_0-PadK4) -> /FPGA_SPARTAN_7/CONFIG/TDO_FPGA
- IC1 pad K5: unconnected-(IC1-TMS_0-PadK5) -> /FPGA_SPARTAN_7/CONFIG/TMS
- IC1 pad K6: unconnected-(IC1-GND_20-PadK6) -> /FPGA_SPARTAN_7/POWER/GND
- IC1 pad K7: unconnected-(IC1-VCCINT_7-PadK7) -> /FPGA_SPARTAN_7/POWER/VCC1V0
- IC1 pad K8: unconnected-(IC1-GND_21-PadK8) -> /FPGA_SPARTAN_7/POWER/GND
- IC1 pad K9: unconnected-(IC1-VCCINT_8-PadK9) -> /FPGA_SPARTAN_7/POWER/VCC1V0
- IC1 pad L11: unconnected-(IC1-IO_L6P_T0_FCS_B_14-PadL11) -> /FPGA_SPARTAN_7/CONFIG/QSPI_CS
- IC1 pad L12: unconnected-(IC1-IO_L6N_T0_D08_VREF_14-PadL12) -> /FPGA_SPARTAN_7/BANK_14/UART_RXD_OUT
- IC1 pad L13: unconnected-(IC1-IO_L7P_T1_D09_14-PadL13) -> /FPGA_SPARTAN_7/BANK_14/PIO29
- IC1 pad L14: unconnected-(IC1-IO_L7N_T1_D10_14-PadL14) -> /FPGA_SPARTAN_7/BANK_14/PIO26
- IC1 pad L15: unconnected-(IC1-IO_L4N_T0_D05_14-PadL15) -> /FPGA_SPARTAN_7/BANK_14/PIO23
- IC1 pad L2: unconnected-(IC1-GND_23-PadL2) -> /FPGA_SPARTAN_7/POWER/GND
- IC1 pad L3: unconnected-(IC1-VCCO_34_3-PadL3) -> /FPGA_SPARTAN_7/POWER/VCC3V3
- IC1 pad L4: unconnected-(IC1-TDI_0-PadL4) -> /FPGA_SPARTAN_7/CONFIG/TDI_FPGA
- IC1 pad L5: unconnected-(IC1-INIT_B_0-PadL5) -> /FPGA_SPARTAN_7/CONFIG/INIT
- IC1 pad L6: unconnected-(IC1-VCCAUX_1-PadL6) -> /FPGA_SPARTAN_7/POWER/VCC1V8
- IC1 pad L7: unconnected-(IC1-GND_24-PadL7) -> /FPGA_SPARTAN_7/POWER/GND
- IC1 pad L8: unconnected-(IC1-VCCAUX_2-PadL8) -> /FPGA_SPARTAN_7/POWER/VCC1V8
- IC1 pad L9: unconnected-(IC1-GND_25-PadL9) -> /FPGA_SPARTAN_7/POWER/GND
- IC1 pad M11: unconnected-(IC1-GND_26-PadM11) -> /FPGA_SPARTAN_7/POWER/GND
- IC1 pad M12: unconnected-(IC1-VCCO_14_2-PadM12) -> /FPGA_SPARTAN_7/POWER/VCC3V3
- IC1 pad M13: unconnected-(IC1-IO_L8P_T1_D11_14-PadM13) -> /FPGA_SPARTAN_7/BANK_14/PIO30
- IC1 pad M14: unconnected-(IC1-IO_L9P_T1_DQS_14-PadM14) -> /FPGA_SPARTAN_7/BANK_14/PIO22
- IC1 pad M15: unconnected-(IC1-IO_L9N_T1_DQS_D13_14-PadM15) -> /FPGA_SPARTAN_7/BANK_14/PIO21
- IC1 pad M5: unconnected-(IC1-M0_0-PadM5) -> /FPGA_SPARTAN_7/CONFIG/MODE_0
- IC1 pad M6: unconnected-(IC1-M2_0-PadM6) -> /FPGA_SPARTAN_7/CONFIG/MODE_2
- IC1 pad M9: unconnected-(IC1-IO_L13P_T2_MRCC_14-PadM9) -> /FPGA_SPARTAN_7/BANK_14/GCLK
- IC1 pad N13: unconnected-(IC1-IO_L8N_T1_D12_14-PadN13) -> /FPGA_SPARTAN_7/BANK_14/PIO18
- IC1 pad N14: unconnected-(IC1-IO_L10P_T1_D14_14-PadN14) -> /FPGA_SPARTAN_7/BANK_14/PIO20
- IC1 pad N15: unconnected-(IC1-IO_L10N_T1_D15_14-PadN15) -> /FPGA_SPARTAN_7/BANK_14/PIO19
- IC1 pad N5: unconnected-(IC1-M1_0-PadN5) -> /FPGA_SPARTAN_7/CONFIG/MODE_1
- IC1 pad P13: unconnected-(IC1-GND_29-PadP13) -> /FPGA_SPARTAN_7/POWER/GND
- IC1 pad P14: unconnected-(IC1-IO_L11P_T1_SRCC_14-PadP14) -> /FPGA_SPARTAN_7/BANK_14/PIO16
- IC1 pad P15: unconnected-(IC1-IO_L11N_T1_SRCC_14-PadP15) -> /FPGA_SPARTAN_7/BANK_14/PIO17
- IC1 pad P4: unconnected-(IC1-GND_27-PadP4) -> /FPGA_SPARTAN_7/POWER/GND
- IC1 pad P5: unconnected-(IC1-VCCO_0_2-PadP5) -> /FPGA_SPARTAN_7/POWER/VCC3V3
- IC1 pad P8: unconnected-(IC1-GND_28-PadP8) -> /FPGA_SPARTAN_7/POWER/GND
- IC1 pad P9: unconnected-(IC1-VCCO_14_3-PadP9) -> /FPGA_SPARTAN_7/POWER/VCC3V3
- IC1 pad R1: unconnected-(IC1-GND_30-PadR1) -> /FPGA_SPARTAN_7/POWER/GND
- IC1 pad R15: unconnected-(IC1-GND_31-PadR15) -> /FPGA_SPARTAN_7/POWER/GND

Commit message: schematic updated
Parts:
- added C10: 4.7uf, Capacitor_SMD:C_0402_1005Metric_Pad0.74x0.62mm_HandSolder, F.Cu at (35.6, -34.0)
- added C11: 4.7uf, Capacitor_SMD:C_0402_1005Metric_Pad0.74x0.62mm_HandSolder, F.Cu at (35.6, -32.0)
- added C12: 47nf, Capacitor_SMD:C_0402_1005Metric_Pad0.74x0.62mm_HandSolder, F.Cu at (35.6, -30.0)
- added C13: 47nf, Capacitor_SMD:C_0402_1005Metric_Pad0.74x0.62mm_HandSolder, F.Cu at (35.6, -28.1)
- added C14: 47nf, Capacitor_SMD:C_0402_1005Metric_Pad0.74x0.62mm_HandSolder, F.Cu at (35.6, -26.1)
- added C15: 47nf, Capacitor_SMD:C_0402_1005Metric_Pad0.74x0.62mm_HandSolder, F.Cu at (38.8, -39.9)
- added C16: 470nf, Capacitor_SMD:C_0402_1005Metric_Pad0.74x0.62mm_HandSolder, F.Cu at (38.8, -37.9)
- added C17: 470nf, Capacitor_SMD:C_0402_1005Metric_Pad0.74x0.62mm_HandSolder, F.Cu at (38.8, -36.0)
- added C18: 4.7uf, Capacitor_SMD:C_0402_1005Metric_Pad0.74x0.62mm_HandSolder, F.Cu at (38.8, -34.0)
- added C19: 47nf, Capacitor_SMD:C_0402_1005Metric_Pad0.74x0.62mm_HandSolder, F.Cu at (38.8, -32.0)
- added C20: 470nf, Capacitor_SMD:C_0402_1005Metric_Pad0.74x0.62mm_HandSolder, F.Cu at (38.8, -30.0)
- added C21: 47nf, Capacitor_SMD:C_0402_1005Metric_Pad0.74x0.62mm_HandSolder, F.Cu at (38.8, -28.1)
- added C22: 47nf, Capacitor_SMD:C_0402_1005Metric_Pad0.74x0.62mm_HandSolder, F.Cu at (38.8, -26.1)
- added C23: 470nf, Capacitor_SMD:C_0402_1005Metric_Pad0.74x0.62mm_HandSolder, F.Cu at (42.0, -39.9)
- added C24: 470nf, Capacitor_SMD:C_0402_1005Metric_Pad0.74x0.62mm_HandSolder, F.Cu at (42.0, -37.9)
- added C25: 470nf, Capacitor_SMD:C_0402_1005Metric_Pad0.74x0.62mm_HandSolder, F.Cu at (42.0, -36.0)
- added C26: 470nf, Capacitor_SMD:C_0402_1005Metric_Pad0.74x0.62mm_HandSolder, F.Cu at (42.0, -34.0)
- added C27: 4.7uf, Capacitor_SMD:C_0402_1005Metric_Pad0.74x0.62mm_HandSolder, F.Cu at (42.0, -32.0)
- added C28: 4.7uf, Capacitor_SMD:C_0402_1005Metric_Pad0.74x0.62mm_HandSolder, F.Cu at (42.0, -30.0)
- added C29: 100uf, Capacitor_SMD:C_0402_1005Metric_Pad0.74x0.62mm_HandSolder, F.Cu at (42.0, -28.1)
- added C30: 47nf, Capacitor_SMD:C_0402_1005Metric_Pad0.74x0.62mm_HandSolder, F.Cu at (42.0, -26.1)
- added C31: 47nf, Capacitor_SMD:C_0402_1005Metric_Pad0.74x0.62mm_HandSolder, F.Cu at (45.2, -39.9)
- added C32: 470nf, Capacitor_SMD:C_0402_1005Metric_Pad0.74x0.62mm_HandSolder, F.Cu at (45.2, -37.9)
- added C33: 470nf, Capacitor_SMD:C_0402_1005Metric_Pad0.74x0.62mm_HandSolder, F.Cu at (45.2, -36.0)
- added C34: 470nf, Capacitor_SMD:C_0402_1005Metric_Pad0.74x0.62mm_HandSolder, F.Cu at (45.2, -34.0)
- added C35: 470nf, Capacitor_SMD:C_0402_1005Metric_Pad0.74x0.62mm_HandSolder, F.Cu at (45.2, -32.0)
- added C36: 47nf, Capacitor_SMD:C_0402_1005Metric_Pad0.74x0.62mm_HandSolder, F.Cu at (45.2, -30.0)
- added C37: 47nf, Capacitor_SMD:C_0402_1005Metric_Pad0.74x0.62mm_HandSolder, F.Cu at (45.2, -28.1)
- added C38: 470nf, Capacitor_SMD:C_0402_1005Metric_Pad0.74x0.62mm_HandSolder, F.Cu at (45.2, -26.1)
- added C39: 470nf, Capacitor_SMD:C_0402_1005Metric_Pad0.74x0.62mm_HandSolder, F.Cu at (48.4, -39.9)
- added C40: 470nf, Capacitor_SMD:C_0402_1005Metric_Pad0.74x0.62mm_HandSolder, F.Cu at (48.4, -37.9)
- added C41: 470nf, Capacitor_SMD:C_0402_1005Metric_Pad0.74x0.62mm_HandSolder, F.Cu at (48.4, -36.0)
- added C42: 4.7uf, Capacitor_SMD:C_0402_1005Metric_Pad0.74x0.62mm_HandSolder, F.Cu at (48.4, -34.0)
- added C43: 4.7uf, Capacitor_SMD:C_0402_1005Metric_Pad0.74x0.62mm_HandSolder, F.Cu at (48.4, -32.0)
- added C44: 100nf, Capacitor_SMD:C_0402_1005Metric_Pad0.74x0.62mm_HandSolder, F.Cu at (63.7, -20.1)
- added C45: 22uf, Capacitor_SMD:C_0402_1005Metric_Pad0.74x0.62mm_HandSolder, F.Cu at (56.9, -39.9)
- added C46: 100NF, Capacitor_SMD:C_0402_1005Metric_Pad0.74x0.62mm_HandSolder, F.Cu at (56.9, -37.9)
- added C47: 20pF, Capacitor_SMD:C_0402_1005Metric_Pad0.74x0.62mm_HandSolder, F.Cu at (56.9, -36.0)
- added C48: 22uf, Capacitor_SMD:C_0402_1005Metric_Pad0.74x0.62mm_HandSolder, F.Cu at (56.9, -34.0)
- added C49: 20pF, Capacitor_SMD:C_0402_1005Metric_Pad0.74x0.62mm_HandSolder, F.Cu at (56.9, -32.0)
- added C50: 10uf, Capacitor_SMD:C_0402_1005Metric_Pad0.74x0.62mm_HandSolder, F.Cu at (56.9, -30.0)
- added C51: 20pF, Capacitor_SMD:C_0402_1005Metric_Pad0.74x0.62mm_HandSolder, F.Cu at (56.9, -28.1)
- added C52: 10uf, Capacitor_SMD:C_0402_1005Metric_Pad0.74x0.62mm_HandSolder, F.Cu at (56.9, -26.1)
- added C53: 12pf, Capacitor_SMD:C_0402_1005Metric_Pad0.74x0.62mm_HandSolder, F.Cu at (38.8, -22.1)
- added C54: 12pf, Capacitor_SMD:C_0402_1005Metric_Pad0.74x0.62mm_HandSolder, F.Cu at (38.8, -20.2)
- added C55: 4.7uf, Capacitor_SMD:C_0402_1005Metric_Pad0.74x0.62mm_HandSolder, F.Cu at (38.8, -18.2)
- added C56: 4.7uf, Capacitor_SMD:C_0402_1005Metric_Pad0.74x0.62mm_HandSolder, F.Cu at (38.8, -16.2)
- added C57: 4.7uf, Capacitor_SMD:C_0402_1005Metric_Pad0.74x0.62mm_HandSolder, F.Cu at (38.8, -14.3)
- added C58: 100nf, Capacitor_SMD:C_0402_1005Metric_Pad0.74x0.62mm_HandSolder, F.Cu at (38.8, -12.3)
- added C59: 100nf, Capacitor_SMD:C_0402_1005Metric_Pad0.74x0.62mm_HandSolder, F.Cu at (38.8, -10.3)
- added C60: 100nf, Capacitor_SMD:C_0402_1005Metric_Pad0.74x0.62mm_HandSolder, F.Cu at (42.1, -22.1)
- added C61: 100nf, Capacitor_SMD:C_0402_1005Metric_Pad0.74x0.62mm_HandSolder, F.Cu at (42.1, -20.2)
- added C62: 100nf, Capacitor_SMD:C_0402_1005Metric_Pad0.74x0.62mm_HandSolder, F.Cu at (42.1, -18.2)
- added C63: 100nf, Capacitor_SMD:C_0402_1005Metric_Pad0.74x0.62mm_HandSolder, F.Cu at (42.1, -16.2)
- added C64: 100nf, Capacitor_SMD:C_0402_1005Metric_Pad0.74x0.62mm_HandSolder, F.Cu at (42.1, -14.3)
- added C65: 100nf, Capacitor_SMD:C_0402_1005Metric_Pad0.74x0.62mm_HandSolder, F.Cu at (42.1, -12.3)
- added C66: 1uf, Capacitor_SMD:C_0402_1005Metric_Pad0.74x0.62mm_HandSolder, F.Cu at (42.1, -10.3)
- added C67: 100nf, Capacitor_SMD:C_0402_1005Metric_Pad0.74x0.62mm_HandSolder, F.Cu at (45.3, -22.1)
- added C68: 100nf, Capacitor_SMD:C_0402_1005Metric_Pad0.74x0.62mm_HandSolder, F.Cu at (45.3, -20.2)
- added C69: 4.7uf, Capacitor_SMD:C_0402_1005Metric_Pad0.74x0.62mm_HandSolder, F.Cu at (45.3, -18.2)
- added C7: 4.7uf, Capacitor_SMD:C_0402_1005Metric_Pad0.74x0.62mm_HandSolder, F.Cu at (35.6, -39.9)
- added C70: 100nf, Capacitor_SMD:C_0402_1005Metric_Pad0.74x0.62mm_HandSolder, F.Cu at (45.3, -16.2)
- added C8: 470nf, Capacitor_SMD:C_0402_1005Metric_Pad0.74x0.62mm_HandSolder, F.Cu at (35.6, -37.9)
- added C9: 470nf, Capacitor_SMD:C_0402_1005Metric_Pad0.74x0.62mm_HandSolder, F.Cu at (35.6, -36.0)
- added D1: LED_Small, LED_SMD:LED_0402_1005Metric_Pad0.77x0.64mm_HandSolder, F.Cu at (64.0, -22.1)
- added D2: PMEG2020EJ,115, Diode_SMD:D_SOD-323F, F.Cu at (103.2, -20.6)
- added D3: BZX84-B2V7,215, SamacSys_Parts:BZX84B2V7215, F.Cu at (98.7, -12.8)
- added D4: LED_Small, LED_SMD:LED_0402_1005Metric_Pad0.77x0.64mm_HandSolder, F.Cu at (60.4, -27.9)
- added D5: LED_Small, LED_SMD:LED_0402_1005Metric_Pad0.77x0.64mm_HandSolder, F.Cu at (48.7, -22.1)
- added D6: LED_Small, LED_SMD:LED_0402_1005Metric_Pad0.77x0.64mm_HandSolder, F.Cu at (48.7, -20.1)
- added D7: LRB520G-30T1G, SamacSys_Parts:BZX84B2V7215, F.Cu at (105.0, -39.0)
- added IC3: MBT3904DW1T1G, SamacSys_Parts:SOT65P210X110-6N, F.Cu at (93.0, -11.0)
- added IC4: 74AHCT125BQ-Q100,1, SamacSys_Parts:74AHCT125BQQ1001, F.Cu at (94.3, -27.3)
- added IC5: M74VHC1GT04DTT1G, SamacSys_Parts:SOT95P275X110-5N, F.Cu at (104.7, -33.8)
- added Q1: SI2302CDS-T1-E3, SamacSys_Parts:SOT95P237X112-3N, F.Cu at (93.2, -19.7)
- added Q2: MMBT4403LT3G, SamacSys_Parts:SOT96P237X111-3N, F.Cu at (93.2, -15.2)
- added R1: 0, Resistor_SMD:R_0402_1005Metric_Pad0.72x0.64mm_HandSolder, F.Cu at (51.7, -39.9)
- added R10: 100, Resistor_SMD:R_0402_1005Metric_Pad0.72x0.64mm_HandSolder, F.Cu at (57.2, -20.1)
- added R11: 100, Resistor_SMD:R_0402_1005Metric_Pad0.72x0.64mm_HandSolder, F.Cu at (57.2, -18.1)
- added R12: 100, Resistor_SMD:R_0402_1005Metric_Pad0.72x0.64mm_HandSolder, F.Cu at (57.2, -16.2)
- added R13: 4.7K, Resistor_SMD:R_0402_1005Metric_Pad0.72x0.64mm_HandSolder, F.Cu at (57.2, -14.2)
- added R14: 4.7K, Resistor_SMD:R_0402_1005Metric_Pad0.72x0.64mm_HandSolder, F.Cu at (57.2, -12.2)
- added R15: 4.7K, Resistor_SMD:R_0402_1005Metric_Pad0.72x0.64mm_HandSolder, F.Cu at (60.5, -22.1)
- added R16: 1.8K, Resistor_SMD:R_0402_1005Metric_Pad0.72x0.64mm_HandSolder, F.Cu at (60.5, -20.1)
- added R17: 1.8K, Resistor_SMD:R_0402_1005Metric_Pad0.72x0.64mm_HandSolder, F.Cu at (60.5, -18.1)
- added R18: 200, Resistor_SMD:R_0402_1005Metric_Pad0.72x0.64mm_HandSolder, F.Cu at (60.5, -16.2)
- added R19: 100, Resistor_SMD:R_0402_1005Metric_Pad0.72x0.64mm_HandSolder, F.Cu at (60.5, -14.2)
- added R2: 0, Resistor_SMD:R_0402_1005Metric_Pad0.72x0.64mm_HandSolder, F.Cu at (51.7, -37.9)
- added R20: 49.9, Resistor_SMD:R_0402_1005Metric_Pad0.72x0.64mm_HandSolder, F.Cu at (54.0, -8.18)
- added R21: 3.48K-1%, Resistor_SMD:R_0402_1005Metric_Pad0.72x0.64mm_HandSolder, F.Cu at (60.1, -39.9)
- added R22: 10K, Resistor_SMD:R_0402_1005Metric_Pad0.72x0.64mm_HandSolder, F.Cu at (60.1, -37.9)
- added R23: 0, Resistor_SMD:R_0402_1005Metric_Pad0.72x0.64mm_HandSolder, F.Cu at (60.1, -35.9)
- added R24: 100K, Resistor_SMD:R_0402_1005Metric_Pad0.72x0.64mm_HandSolder, F.Cu at (60.1, -33.9)
- added R25: 30K, Resistor_SMD:R_0402_1005Metric_Pad0.72x0.64mm_HandSolder, F.Cu at (60.1, -31.9)
- added R26: 120K, Resistor_SMD:R_0402_1005Metric_Pad0.72x0.64mm_HandSolder, F.Cu at (60.1, -29.9)
- added R27: 150K, Resistor_SMD:R_0402_1005Metric_Pad0.72x0.64mm_HandSolder, F.Cu at (63.4, -39.9)
- added R28: 120K, Resistor_SMD:R_0402_1005Metric_Pad0.72x0.64mm_HandSolder, F.Cu at (63.4, -37.9)
- added R29: 180K, Resistor_SMD:R_0402_1005Metric_Pad0.72x0.64mm_HandSolder, F.Cu at (63.4, -35.9)
- added R3: 1K, Resistor_SMD:R_0402_1005Metric_Pad0.72x0.64mm_HandSolder, F.Cu at (54.0, -22.1)
- added R30: 57.6K, Resistor_SMD:R_0402_1005Metric_Pad0.72x0.64mm_HandSolder, F.Cu at (63.4, -33.9)
- added R31: 100K, Resistor_SMD:R_0402_1005Metric_Pad0.72x0.64mm_HandSolder, F.Cu at (63.4, -31.9)
- added R32: 100K, Resistor_SMD:R_0402_1005Metric_Pad0.72x0.64mm_HandSolder, F.Cu at (63.4, -29.9)
- added R33: 1K, Resistor_SMD:R_0402_1005Metric_Pad0.72x0.64mm_HandSolder, F.Cu at (66.6, -39.9)
- added R34: 120, Resistor_SMD:R_0402_1005Metric_Pad0.72x0.64mm_HandSolder, F.Cu at (66.6, -37.9)
- added R35: 22, Resistor_SMD:R_0402_1005Metric_Pad0.72x0.64mm_HandSolder, F.Cu at (66.6, -35.9)
- added R36: 100K, Resistor_SMD:R_0402_1005Metric_Pad0.72x0.64mm_HandSolder, F.Cu at (66.6, -33.9)
- added R37: 680, Resistor_SMD:R_0402_1005Metric_Pad0.72x0.64mm_HandSolder, F.Cu at (66.6, -31.9)
- added R38: 33, Resistor_SMD:R_0402_1005Metric_Pad0.72x0.64mm_HandSolder, F.Cu at (35.6, -22.1)
- added R39: 33, Resistor_SMD:R_0402_1005Metric_Pad0.72x0.64mm_HandSolder, F.Cu at (35.6, -20.1)
- added R4: 1K, Resistor_SMD:R_0402_1005Metric_Pad0.72x0.64mm_HandSolder, F.Cu at (54.0, -20.1)
- added R40: 33, Resistor_SMD:R_0402_1005Metric_Pad0.72x0.64mm_HandSolder, F.Cu at (35.6, -18.1)
- added R41: 1K, Resistor_SMD:R_0402_1005Metric_Pad0.72x0.64mm_HandSolder, F.Cu at (35.6, -16.2)
- added R42: 12K, Resistor_SMD:R_0402_1005Metric_Pad0.72x0.64mm_HandSolder, F.Cu at (35.6, -14.2)
- added R43: 2.2K, Resistor_SMD:R_0402_1005Metric_Pad0.72x0.64mm_HandSolder, F.Cu at (35.6, -12.2)
- added R44: 2.2K, Resistor_SMD:R_0402_1005Metric_Pad0.72x0.64mm_HandSolder, F.Cu at (35.6, -10.2)
- added R45: 10K, Resistor_SMD:R_0402_1005Metric_Pad0.72x0.64mm_HandSolder, F.Cu at (35.6, -8.19)
- added R5: 1K, Resistor_SMD:R_0402_1005Metric_Pad0.72x0.64mm_HandSolder, F.Cu at (54.0, -18.1)
- added R6: 4.7K, Resistor_SMD:R_0402_1005Metric_Pad0.72x0.64mm_HandSolder, F.Cu at (54.0, -16.2)
- added R7: 49.9K, Resistor_SMD:R_0402_1005Metric_Pad0.72x0.64mm_HandSolder, F.Cu at (54.0, -14.2)
- added R8: 1K, Resistor_SMD:R_0402_1005Metric_Pad0.72x0.64mm_HandSolder, F.Cu at (54.0, -12.2)
- added R9: 100, Resistor_SMD:R_0402_1005Metric_Pad0.72x0.64mm_HandSolder, F.Cu at (57.2, -22.1)
- added U2: FT2232HQ, Package_DFN_QFN:QFN-64-1EP_9x9mm_P0.5mm_EP4.35x4.35mm, F.Cu at (121.2, 75.1)
- added Y1: ABM3B-12.000MHZ-12-N2Y-T, SamacSys_Parts:ABM3B, F.Cu at (101.3, -28.3)
- IC2: value FT2232H-56Q-TRAY -> LTC3569EUDC#PBF; footprint SamacSys_Parts:QFN50P800X800X100-57N-D -> SamacSys_Parts:QFN50P300X400X80-21N-D
- moved IC2 84.0 mm to (98.4, -18.9)
- moved IC1 41.3 mm to (150.0, 75.0)
- moved U1 11.0 mm to (131.6, 62.2)
Connections:
- net /FPGA_SPARTAN_7/POWER/VCC1V0 renamed /FPGA_SPARTAN_7/VCC1V0
- net /FPGA_SPARTAN_7/POWER/VCC1V8 renamed /FPGA_SPARTAN_7/VCC1V8
- IC1 pad A1: /FPGA_SPARTAN_7/POWER/GND -> GND
- IC1 pad A15: /FPGA_SPARTAN_7/POWER/GND -> GND
- IC1 pad B8: /FPGA_SPARTAN_7/POWER/GND -> GND
- IC1 pad C12: /FPGA_SPARTAN_7/POWER/GND -> GND
- IC1 pad C2: /FPGA_SPARTAN_7/POWER/GND -> GND
- IC1 pad C3: /FPGA_SPARTAN_7/POWER/VCC3V3 -> /FPGA_SPARTAN_7/VCC3V3
- IC1 pad D14: /FPGA_SPARTAN_7/POWER/GND -> GND
- IC1 pad D6: /FPGA_SPARTAN_7/POWER/GND -> GND
- IC1 pad E4: /FPGA_SPARTAN_7/POWER/GND -> GND
- IC1 pad E5: /FPGA_SPARTAN_7/CONFIG/TCLK -> /FPGA_SPARTAN_7/TCLK
- IC1 pad E6: /FPGA_SPARTAN_7/POWER/VCC3V3 -> /FPGA_SPARTAN_7/VCC3V3
- IC1 pad E7: /FPGA_SPARTAN_7/POWER/GND -> GND
- IC1 pad E9: /FPGA_SPARTAN_7/POWER/GND -> GND
- IC1 pad F10: /FPGA_SPARTAN_7/POWER/GND -> GND
- IC1 pad F13: /FPGA_SPARTAN_7/POWER/GND -> GND
- IC1 pad F6: /FPGA_SPARTAN_7/POWER/GND -> GND
- IC1 pad G2: /FPGA_SPARTAN_7/POWER/VCC3V3 -> /FPGA_SPARTAN_7/VCC3V3
- IC1 pad G3: /FPGA_SPARTAN_7/POWER/GND -> GND
- IC1 pad G7: /FPGA_SPARTAN_7/POWER/GND -> GND
- IC1 pad H10: /FPGA_SPARTAN_7/POWER/GND -> GND
- IC1 pad H6: /FPGA_SPARTAN_7/POWER/GND -> GND
- IC1 pad J13: /FPGA_SPARTAN_7/POWER/GND -> GND
- IC1 pad J14: /FPGA_SPARTAN_7/POWER/VCC3V3 -> /FPGA_SPARTAN_7/VCC3V3
- IC1 pad J7: /FPGA_SPARTAN_7/POWER/GND -> GND
- IC1 pad K10: /FPGA_SPARTAN_7/POWER/GND -> GND
- IC1 pad K4: /FPGA_SPARTAN_7/CONFIG/TDO_FPGA -> /FPGA_SPARTAN_7/TDO_FPGA
- IC1 pad K5: /FPGA_SPARTAN_7/CONFIG/TMS -> /FPGA_SPARTAN_7/TMS
- IC1 pad K6: /FPGA_SPARTAN_7/POWER/GND -> GND
- IC1 pad K8: /FPGA_SPARTAN_7/POWER/GND -> GND
- IC1 pad L2: /FPGA_SPARTAN_7/POWER/GND -> GND
- IC1 pad L3: /FPGA_SPARTAN_7/POWER/VCC3V3 -> /FPGA_SPARTAN_7/VCC3V3
- IC1 pad L4: /FPGA_SPARTAN_7/CONFIG/TDI_FPGA -> /FPGA_SPARTAN_7/TDI_FPGA
- IC1 pad L7: /FPGA_SPARTAN_7/POWER/GND -> GND
- IC1 pad L9: /FPGA_SPARTAN_7/POWER/GND -> GND
- IC1 pad M11: /FPGA_SPARTAN_7/POWER/GND -> GND
- IC1 pad M12: /FPGA_SPARTAN_7/POWER/VCC3V3 -> /FPGA_SPARTAN_7/VCC3V3
- IC1 pad P13: /FPGA_SPARTAN_7/POWER/GND -> GND
- IC1 pad P4: /FPGA_SPARTAN_7/POWER/GND -> GND
- IC1 pad P5: /FPGA_SPARTAN_7/POWER/VCC3V3 -> /FPGA_SPARTAN_7/VCC3V3
- IC1 pad P8: /FPGA_SPARTAN_7/POWER/GND -> GND
- IC1 pad P9: /FPGA_SPARTAN_7/POWER/VCC3V3 -> /FPGA_SPARTAN_7/VCC3V3
- IC1 pad R1: /FPGA_SPARTAN_7/POWER/GND -> GND
- IC1 pad R15: /FPGA_SPARTAN_7/POWER/GND -> GND
- IC2 pad 1: unconnected-(IC2-EECS-Pad1) -> GND
- IC2 pad 10: unconnected-(IC2-TEST-Pad10) -> /POWER_REGULATOR/VU
- IC2 pad 11: unconnected-(IC2-RESET#-Pad11) -> GND
- IC2 pad 12: unconnected-(IC2-ADBUS0-Pad12) -> Net-(IC2-EN3)
- IC2 pad 13: unconnected-(IC2-ADBUS1-Pad13) -> /POWER_REGULATOR/EN2
- IC2 pad 14: unconnected-(IC2-ADBUS2-Pad14) -> /POWER_REGULATOR/VU
- IC2 pad 15: unconnected-(IC2-ADBUS3-Pad15) -> GND
- IC2 pad 16: unconnected-(IC2-VCCIO_1-Pad16) -> Net-(IC2-SW3)
- IC2 pad 17: unconnected-(IC2-ADBUS4-Pad17) -> /POWER_REGULATOR/VU
- IC2 pad 18: unconnected-(IC2-ADBUS5-Pad18) -> /POWER_REGULATOR/VU
- IC2 pad 19: unconnected-(IC2-ADBUS6-Pad19) -> Net-(IC2-SW1)
- IC2 pad 2: unconnected-(IC2-VCORE_1-Pad2) -> Net-(IC2-SW2)
- IC2 pad 20: unconnected-(IC2-ADBUS7-Pad20) -> GND
- IC2 pad 21: unconnected-(IC2-GND_1-Pad21) -> GND
- IC2 pad 3: unconnected-(IC2-OSCI-Pad3) -> /POWER_REGULATOR/VU
- IC2 pad 4: unconnected-(IC2-OSCO-Pad4) -> /POWER_REGULATOR/PGOOD
- IC2 pad 5: unconnected-(IC2-VPHY-Pad5) -> Net-(IC2-MODE)
- IC2 pad 6: unconnected-(IC2-REF-Pad6) -> /POWER_REGULATOR/VU
- IC2 pad 7: unconnected-(IC2-DM-Pad7) -> Net-(IC2-FB2)
- IC2 pad 8: unconnected-(IC2-DP-Pad8) -> Net-(IC2-FB1)
- IC2 pad 9: unconnected-(IC2-VPLL-Pad9) -> Net-(IC2-FB3)
- U1 pad 8: /FPGA_SPARTAN_7/CONFIG/VCC3V3 -> /FPGA_SPARTAN_7/VCC3V3
Other:
- board outline added: 100 x 50 mm

Commit message: updated schematic
Parts:
- added C71: 10uf, Capacitor_SMD:C_0603_1608Metric, F.Cu at (118.3, 64.4)
- added D10: LESD5D5.0CT1G, SamacSys_Parts:LESD5D50CT1G, F.Cu at (110.4, 75.7)
- added D11: LESD5D5.0CT1G, SamacSys_Parts:LESD5D50CT1G, F.Cu at (108.5, 75.7)
- added D8: LESD5D5.0CT1G, SamacSys_Parts:LESD5D50CT1G, F.Cu at (112.4, 75.7)
- added J1: U254-051N-4BH806, footprints:U254-051N-4BH806, F.Cu at (105.5, 75.0)
- added R46: 0, Resistor_SMD:R_0402_1005Metric_Pad0.72x0.64mm_HandSolder, B.Cu at (112.8, 74.7)
- added R47: 0, Resistor_SMD:R_0402_1005Metric_Pad0.72x0.64mm_HandSolder, B.Cu at (112.7, 75.9)
- added R48: 0, Resistor_SMD:R_0402_1005Metric_Pad0.72x0.64mm_HandSolder, F.Cu at (138.4, 69.3)
- added R49: 0, Resistor_SMD:R_0402_1005Metric_Pad0.72x0.64mm_HandSolder, F.Cu at (138.4, 71.2)
- added R50: 140, Resistor_SMD:R_0402_1005Metric_Pad0.72x0.64mm_HandSolder, F.Cu at (162.4, 59.4)
- added R51: 845, Resistor_SMD:R_0402_1005Metric_Pad0.72x0.64mm_HandSolder, F.Cu at (164.4, 59.4)
- added R52: 140, Resistor_SMD:R_0402_1005Metric_Pad0.72x0.64mm_HandSolder, F.Cu at (166.4, 59.4)
- added R53: 845, Resistor_SMD:R_0402_1005Metric_Pad0.72x0.64mm_HandSolder, F.Cu at (168.4, 59.4)
- added R54: 1K, Resistor_SMD:R_0402_1005Metric_Pad0.72x0.64mm_HandSolder, F.Cu at (170.3, 59.4)
- added R55: 1K, Resistor_SMD:R_0402_1005Metric_Pad0.72x0.64mm_HandSolder, F.Cu at (172.3, 59.4)
- added R56: 2.32K, Resistor_SMD:R_0402_1005Metric_Pad0.72x0.64mm_HandSolder, F.Cu at (174.3, 59.4)
- added R57: 2.32K, Resistor_SMD:R_0402_1005Metric_Pad0.72x0.64mm_HandSolder, F.Cu at (176.3, 59.4)
- C57, C68, C69, C70, R41, R42: moved to B.Cu
- moved C15 163.1 mm to (164.4, 64.1)
- moved C16 163.1 mm to (164.4, 66.1)
- moved C17 163.1 mm to (164.4, 68.0)
- moved C18 163.1 mm to (164.4, 70.0)
- moved C19 163.1 mm to (164.4, 72.0)
- moved C20 163.1 mm to (164.4, 74.0)
- moved C21 163.1 mm to (164.4, 75.9)
- moved C22 163.1 mm to (164.4, 77.9)
- moved C39 163.1 mm to (174.0, 64.1)
- moved C40 163.1 mm to (174.0, 66.1)
- moved C41 163.1 mm to (174.0, 68.0)
- moved C42 163.1 mm to (174.0, 70.0)
- moved C43 163.1 mm to (174.0, 72.0)
- moved C44 163.1 mm to (189.3, 83.8)
- moved C61 163.1 mm to (167.6, 83.8)
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Connections:
- C19 pad 1: /FPGA_SPARTAN_7/VCC3V3 -> +3V3
- C20 pad 1: /FPGA_SPARTAN_7/VCC3V3 -> +3V3
- C21 pad 1: /FPGA_SPARTAN_7/VCC3V3 -> +3V3
- C22 pad 1: /FPGA_SPARTAN_7/VCC3V3 -> +3V3
- C23 pad 1: /FPGA_SPARTAN_7/VCC3V3 -> +3V3
- C24 pad 1: /FPGA_SPARTAN_7/VCC3V3 -> +3V3
- C25 pad 1: /FPGA_SPARTAN_7/VCC3V3 -> +3V3
- C26 pad 1: /FPGA_SPARTAN_7/VCC3V3 -> +3V3
- C27 pad 1: /FPGA_SPARTAN_7/VCC3V3 -> +3V3
- C28 pad 1: /FPGA_SPARTAN_7/VCC3V3 -> +3V3
- C29 pad 1: /FPGA_SPARTAN_7/VCC3V3 -> +3V3
- C36 pad 1: /FPGA_SPARTAN_7/VCC3V3 -> +3V3
- C37 pad 1: /FPGA_SPARTAN_7/VCC3V3 -> +3V3
- C38 pad 1: /FPGA_SPARTAN_7/VCC3V3 -> +3V3
- C39 pad 1: /FPGA_SPARTAN_7/VCC3V3 -> +3V3
- C40 pad 1: /FPGA_SPARTAN_7/VCC3V3 -> +3V3
- C41 pad 1: /FPGA_SPARTAN_7/VCC3V3 -> +3V3
- C42 pad 1: /FPGA_SPARTAN_7/VCC3V3 -> +3V3
- C43 pad 1: /FPGA_SPARTAN_7/VCC3V3 -> +3V3
- C44 pad 1: /FPGA_SPARTAN_7/VCC3V3 -> +3V3
- C51 pad 1: /FPGA_SPARTAN_7/VCC3V3 -> +3V3
- C52 pad 1: /FPGA_SPARTAN_7/VCC3V3 -> +3V3
- C56 pad 1: Net-(U2-VREGIN) -> +3V3
- D4 pad 2: /FPGA_SPARTAN_7/VCC3V3 -> +3V3
- IC1 pad A11: unconnected-(IC1C-IO_L11P_T1_SRCC_AD12P_15-PadA11) -> /FPGA_SPARTAN_7/BANK_15/AIN33_P
- IC1 pad A12: unconnected-(IC1C-IO_L11N_T1_SRCC_AD12N_15-PadA12) -> /FPGA_SPARTAN_7/BANK_15/AIN33_N
- IC1 pad A13: unconnected-(IC1C-IO_L12P_T1_MRCC_AD5P_15-PadA13) -> /FPGA_SPARTAN_7/BANK_15/AIN32_P
- IC1 pad A14: unconnected-(IC1C-IO_L12N_T1_MRCC_AD5N_15-PadA14) -> /FPGA_SPARTAN_7/BANK_15/AIN32_N
- IC1 pad A2: unconnected-(IC1D-IO_L2N_T0_34-PadA2) -> /FPGA_SPARTAN_7/BANK_34/PIO41
- IC1 pad A3: unconnected-(IC1D-IO_L1N_T0_34-PadA3) -> /FPGA_SPARTAN_7/BANK_34/PIO47
- IC1 pad A4: unconnected-(IC1D-IO_L1P_T0_34-PadA4) -> /FPGA_SPARTAN_7/BANK_34/PIO48
- IC1 pad B1: unconnected-(IC1D-IO_L4N_T0_34-PadB1) -> /FPGA_SPARTAN_7/BANK_34/PIO43
- IC1 pad B2: unconnected-(IC1D-IO_L2P_T0_34-PadB2) -> /FPGA_SPARTAN_7/BANK_34/PIO42
- IC1 pad B3: unconnected-(IC1D-IO_L3N_T0_DQS_34-PadB3) -> /FPGA_SPARTAN_7/BANK_34/PIO45
- IC1 pad B4: unconnected-(IC1D-IO_L3P_T0_DQS_34-PadB4) -> /FPGA_SPARTAN_7/BANK_34/PIO46
- IC1 pad C1: unconnected-(IC1D-IO_L4P_T0_34-PadC1) -> /FPGA_SPARTAN_7/BANK_34/PIO44
- IC1 pad C3: /FPGA_SPARTAN_7/VCC3V3 -> +3V3
- IC1 pad C5: unconnected-(IC1D-IO_L5P_T0_34-PadC5) -> /FPGA_SPARTAN_7/BANK_34/PIO40
- IC1 pad D1: unconnected-(IC1D-IO_L6N_T0_VREF_34-PadD1) -> /FPGA_SPARTAN_7/BANK_34/BTN1
- IC1 pad D2: unconnected-(IC1D-IO_L6P_T0_34-PadD2) -> /FPGA_SPARTAN_7/BANK_34/BTN0
- IC1 pad D3: unconnected-(IC1D-IO_L9N_T1_DQS_34-PadD3) -> /FPGA_SPARTAN_7/BANK_34/LED0_G
- IC1 pad E1: unconnected-(IC1D-IO_L8N_T1_34-PadE1) -> /FPGA_SPARTAN_7/BANK_34/LED4
- IC1 pad E2: unconnected-(IC1D-IO_L8P_T1_34-PadE2) -> /FPGA_SPARTAN_7/BANK_34/LED1
- IC1 pad E6: /FPGA_SPARTAN_7/VCC3V3 -> +3V3
- IC1 pad F1: unconnected-(IC1D-IO_L10N_T1_34-PadF1) -> /FPGA_SPARTAN_7/BANK_34/LED0_B
- IC1 pad F2: unconnected-(IC1D-IO_L10P_T1_34-PadF2) -> /FPGA_SPARTAN_7/BANK_34/LED0_R
- IC1 pad F3: unconnected-(IC1D-IO_L11N_T1_SRCC_34-PadF3) -> /FPGA_SPARTAN_7/BANK_34/JA4
- IC1 pad F4: unconnected-(IC1D-IO_L11P_T1_SRCC_34-PadF4) -> /FPGA_SPARTAN_7/BANK_34/JA10
- IC1 pad G1: unconnected-(IC1D-IO_L12N_T1_MRCC_34-PadG1) -> /FPGA_SPARTAN_7/BANK_34/JA9
- IC1 pad G2: /FPGA_SPARTAN_7/VCC3V3 -> +3V3
- IC1 pad H1: unconnected-(IC1D-IO_L12P_T1_MRCC_34-PadH1) -> /FPGA_SPARTAN_7/BANK_34/JA8
- IC1 pad H2: unconnected-(IC1D-IO_L14N_T2_SRCC_34-PadH2) -> /FPGA_SPARTAN_7/BANK_34/JA2
- IC1 pad H3: unconnected-(IC1D-IO_L13N_T2_MRCC_34-PadH3) -> /FPGA_SPARTAN_7/BANK_34/JA7
- IC1 pad H4: unconnected-(IC1D-IO_L13P_T2_MRCC_34-PadH4) -> /FPGA_SPARTAN_7/BANK_34/JA3
- IC1 pad J1: unconnected-(IC1D-IO_L16N_T2_34-PadJ1) -> /FPGA_SPARTAN_7/BANK_34/LED3
- IC1 pad J14: /FPGA_SPARTAN_7/VCC3V3 -> +3V3
- IC1 pad J2: unconnected-(IC1D-IO_L14P_T2_SRCC_34-PadJ2) -> /FPGA_SPARTAN_7/BANK_34/JA1
- IC1 pad K1: unconnected-(IC1D-IO_L16P_T2_34-PadK1) -> /FPGA_SPARTAN_7/BANK_34/LED1
- IC1 pad K15: /FPGA_SPARTAN_7/BANK_14/UART_TXD_IN -> /FPGA_SPARTAN_7/BANK_14/UART_RXD_OUT
- IC1 pad L1: unconnected-(IC1D-IO_L18N_T2_34-PadL1) -> /FPGA_SPARTAN_7/BANK_34/PIO01
- IC1 pad L3: /FPGA_SPARTAN_7/VCC3V3 -> +3V3
- IC1 pad M12: /FPGA_SPARTAN_7/VCC3V3 -> +3V3
- IC1 pad M2: unconnected-(IC1D-IO_L20N_T3_34-PadM2) -> /FPGA_SPARTAN_7/BANK_34/PIO05
- IC1 pad M3: unconnected-(IC1D-IO_L19N_T3_VREF_34-PadM3) -> /FPGA_SPARTAN_7/BANK_34/PIO03
- IC1 pad M4: unconnected-(IC1D-IO_L19P_T3_34-PadM4) -> /FPGA_SPARTAN_7/BANK_34/PIO02
- IC1 pad N1: unconnected-(IC1D-IO_L22N_T3_34-PadN1) -> /FPGA_SPARTAN_7/BANK_34/PIO09
- IC1 pad N2: unconnected-(IC1D-IO_L20P_T3_34-PadN2) -> /FPGA_SPARTAN_7/BANK_34/PIO04
- IC1 pad N3: unconnected-(IC1D-IO_L21N_T3_DQS_34-PadN3) -> /FPGA_SPARTAN_7/BANK_34/PIO07
- IC1 pad P1: unconnected-(IC1D-IO_L22P_T3_34-PadP1) -> /FPGA_SPARTAN_7/BANK_34/PIO08
- IC1 pad P3: unconnected-(IC1D-IO_L21P_T3_DQS_34-PadP3) -> /FPGA_SPARTAN_7/BANK_34/PIO06
- IC1 pad P5: /FPGA_SPARTAN_7/VCC3V3 -> +3V3
- IC1 pad P9: /FPGA_SPARTAN_7/VCC3V3 -> +3V3
- Q2 pad 2: /FPGA_SPARTAN_7/VCC3V3 -> +3V3
- R13 pad 2: /FPGA_SPARTAN_7/VCC3V3 -> +3V3
- R14 pad 2: /FPGA_SPARTAN_7/VCC3V3 -> +3V3
- R15 pad 2: /FPGA_SPARTAN_7/VCC3V3 -> +3V3
- R16 pad 2: /FPGA_SPARTAN_7/VCC3V3 -> +3V3
- R17 pad 2: /FPGA_SPARTAN_7/VCC3V3 -> +3V3
- R18 pad 2: /FPGA_SPARTAN_7/VCC3V3 -> +3V3
- R2 pad 2: /FPGA_SPARTAN_7/VCC3V3 -> +3V3
- R29 pad 1: /FPGA_SPARTAN_7/VCC3V3 -> +3V3
- R34 pad 1: /FPGA_SPARTAN_7/VCC3V3 -> +3V3
- R36 pad 1: /FPGA_SPARTAN_7/VCC3V3 -> +3V3
- R8 pad 1: /FPGA_SPARTAN_7/VCC3V3 -> +3V3
- U1 pad 8: /FPGA_SPARTAN_7/VCC3V3 -> +3V3
- U2 pad 50: Net-(U2-VREGIN) -> +3V3
Routing:
- net /POWER_REGULATOR/USB5V0: track 0.00 -> 8.12 mm
- net Net-(D10-A2): track 0.00 -> 5.43 mm
- net Net-(D11-A2): track 0.00 -> 2.98 mm
Other:
- outline, holes or cut-outs redrawn
- copper layers 2 -> 6
