File: kicad_files/sparton_7.kicad_pcb (KiCad board)
At the start: 6 copper layers, 75 x 50 mm, 185 parts, among them IC1 XC7S25-1CSGA225C, IC2 LTC3569EUDC#PBF, IC3 MBT3904DW1T1G, IC4 74AHCT125BQ-Q100,1, IC5 M74VHC1GT04DTT1G, IC6 M93C46-WMN6TP, J1 U254-051N-4BH806, J2 Conn_02x10_Odd_Even, J3 Conn_02x05_Odd_Even, J4 Conn_02x06_Odd_Even, Q1 SI2302CDS-T1-E3, Q2 MMBT4403LT3G, U1 MX25L3233FM2I-08G, U2 FT2232HQ, Y1 ABM3B-12.000MHZ-12-N2Y-T

Commit message: updated files
Parts:
- moved FB2 0.57 mm to (148.0, 72.3)
- moved C20 0.37 mm to (150.2, 70.6), turned to 0 degrees
- moved C2 0.12 mm to (146.5, 73.0)
- turned J3 to -90 degrees
Connections:
- C10 pad 1: /FPGA_SPARTAN_7/VCC1V8 -> +1V8
- C11 pad 1: /FPGA_SPARTAN_7/VCC1V8 -> +1V8
- C12 pad 1: /FPGA_SPARTAN_7/VCC1V8 -> +1V8
- C13 pad 1: /FPGA_SPARTAN_7/VCC1V8 -> +1V8
- C49 pad 1: /FPGA_SPARTAN_7/VCC1V8 -> +1V8
- C50 pad 1: /FPGA_SPARTAN_7/VCC1V8 -> +1V8
- C8 pad 1: /FPGA_SPARTAN_7/VCC1V8 -> +1V8
- C9 pad 1: /FPGA_SPARTAN_7/VCC1V8 -> +1V8
- FB2 pad 2: /FPGA_SPARTAN_7/VCC1V8 -> +1V8
- IC1 pad L6: /FPGA_SPARTAN_7/VCC1V8 -> +1V8
- IC1 pad L8: /FPGA_SPARTAN_7/VCC1V8 -> +1V8
- J3 pad 1: /FPGA_SPARTAN_7/BANK_15/AIN33 -> /FPGA_SPARTAN_7/BANK_34/JA7
- J3 pad 10: /FPGA_SPARTAN_7/BANK_34/JA7 -> /FPGA_SPARTAN_7/BANK_15/AIN33
- J3 pad 2: /FPGA_SPARTAN_7/BANK_34/JA1 -> /FPGA_SPARTAN_7/BANK_34/JA8
- J3 pad 3: /FPGA_SPARTAN_7/BANK_15/AIN32 -> /FPGA_SPARTAN_7/BANK_34/JA4
- J3 pad 4: /FPGA_SPARTAN_7/BANK_34/JA2 -> /FPGA_SPARTAN_7/BANK_34/JA9
- J3 pad 5: /FPGA_SPARTAN_7/BANK_34/JA10 -> /FPGA_SPARTAN_7/BANK_34/JA3
- J3 pad 6: /FPGA_SPARTAN_7/BANK_34/JA3 -> /FPGA_SPARTAN_7/BANK_34/JA10
- J3 pad 7: /FPGA_SPARTAN_7/BANK_34/JA9 -> /FPGA_SPARTAN_7/BANK_34/JA2
- J3 pad 8: /FPGA_SPARTAN_7/BANK_34/JA4 -> /FPGA_SPARTAN_7/BANK_15/AIN32
- J3 pad 9: /FPGA_SPARTAN_7/BANK_34/JA8 -> /FPGA_SPARTAN_7/BANK_34/JA1
- L2 pad 2: /FPGA_SPARTAN_7/VCC1V8 -> +1V8
- R1 pad 2: /FPGA_SPARTAN_7/VCC1V8 -> +1V8
- R21 pad 1: /FPGA_SPARTAN_7/VCC1V8 -> +1V8
- R27 pad 1: /FPGA_SPARTAN_7/VCC1V8 -> +1V8
Routing:
- net +1V8: track 8.68 -> 175.6 mm, vias 0 -> 19
- net /FPGA_SPARTAN_7/VCC1V8: track 36.6 -> 0.00 mm, vias 2 -> 0
- net GND: track 94.9 -> 114.3 mm, vias 92 -> 105
- net /POWER_REGULATOR/VU: track 44.1 -> 49.6 mm
- net Net-(IC6-DU): track 0.00 -> 1.73 mm
- added copper zone on F.Cu, net +1V8
