File: kicad_files/FPGA_SPARTAN_7.kicad_sch (KiCad schematic)
At the start: 0 parts

Commit message: ftdi progess
Changed lines of the file:
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@@
     )
   )
-  (sheet (at 119.38 105.41) (size 53.975 60.325) (fields_autoplaced)
+  (sheet (at 119.38 107.315) (size 53.975 60.325) (fields_autoplaced)
     (stroke (width 0.1524) (type solid))
     (fill (color 0 0 0 0.0000))
-    (property "Sheetname" "BANK_34" (at 119.38 104.6984 0)
+    (property "Sheetname" "BANK_34" (at 119.38 106.6034 0)
       (effects (font (size 1.27 1.27)) (justify left bottom))
     )
-    (property "Sheetfile" "BANK_34.kicad_sch" (at 119.38 166.3196 0)
+    (property "Sheetfile" "BANK_34.kicad_sch" (at 119.38 168.2246 0)
       (effects (font (size 1.27 1.27)) (justify left top))
     )
-    (property "Field2" "" (at 119.38 105.41 0)
+    (property "Field2" "" (at 119.38 107.315 0)
       (effects (font (size 1.27 1.27)) hide)
     )
@@
     )
   )
-  (sheet (at 202.565 30.48) (size 53.975 60.325) (fields_autoplaced)
+  (sheet (at 202.565 32.385) (size 53.975 60.325) (fields_autoplaced)
     (stroke (width 0.1524) (type solid))
     (fill (color 0 0 0 0.0000))
-    (property "Sheetname" "BANK_14" (at 202.565 29.7684 0)
+    (property "Sheetname" "BANK_14" (at 202.565 31.6734 0)
       (effects (font (size 1.27 1.27)) (justify left bottom))
     )
-    (property "Sheetfile" "BANK_14.kicad_sch" (at 202.565 91.3896 0)
+    (property "Sheetfile" "BANK_14.kicad_sch" (at 202.565 93.2946 0)
       (effects (font (size 1.27 1.27)) (justify left top))
     )
-    (property "Field2" "" (at 202.565 30.48 0)
+    (property "Field2" "" (at 202.565 32.385 0)
       (effects (font (size 1.27 1.27)) hide)
     )
@@
     )
   )
-  (sheet (at 38.735 107.315) (size 53.975 60.325) (fields_autoplaced)
+  (sheet (at 35.56 107.315) (size 53.975 60.325) (fields_autoplaced)
     (stroke (width 0.1524) (type solid))
     (fill (color 0 0 0 0.0000))
-    (property "Sheetname" "BANK_15" (at 38.735 106.6034 0)
+    (property "Sheetname" "BANK_15" (at 35.56 106.6034 0)
       (effects (font (size 1.27 1.27)) (justify left bottom))
     )
-    (property "Sheetfile" "BANK_15.kicad_sch" (at 38.735 168.2246 0)
+    (property "Sheetfile" "BANK_15.kicad_sch" (at 35.56 168.2246 0)
       (effects (font (size 1.27 1.27)) (justify left top))
     )
-    (property "Field2" "" (at 38.735 107.315 0)
+    (property "Field2" "" (at 35.56 107.315 0)
       (effects (font (size 1.27 1.27)) hide)
     )

Commit message: schematic updated
Other:
- sheet CONFIG ports: added TCLK, TDI_FPGA, TDO_FPGA, TMS, VCC3V3; removed none
- sheet POWER ports: added VCC1V0, VCC1V8, VCC3V3; removed none
Changed lines of the file:
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@@
 (kicad_sch (version 20230121) (generator eeschema)
   (paper "A4")
+  (junction (at 65.405 19.685) (diameter 0) (color 0 0 0 0)
+  )
+  (wire (pts (xy 65.405 19.685) (xy 65.405 32.385))
+    (stroke (width 0) (type default))
+  )
+  (wire (pts (xy 150.495 32.385) (xy 150.495 24.765))
+    (stroke (width 0) (type default))
+  )
+  (wire (pts (xy 147.955 21.59) (xy 162.56 21.59))
+    (stroke (width 0) (type default))
+  )
+  (wire (pts (xy 55.245 32.385) (xy 55.245 19.685))
+    (stroke (width 0) (type default))
+  )
+  (wire (pts (xy 44.45 17.145) (xy 60.325 17.145))
+    (stroke (width 0) (type default))
+  )
+  (wire (pts (xy 138.43 19.685) (xy 138.43 32.385))
+    (stroke (width 0) (type default))
+  )
+  (wire (pts (xy 144.78 32.385) (xy 144.78 18.415))
+    (stroke (width 0) (type default))
+  )
+  (wire (pts (xy 68.58 15.875) (xy 65.405 15.875))
+    (stroke (width 0) (type default))
+  )
+  (wire (pts (xy 60.325 32.385) (xy 60.325 17.145))
+    (stroke (width 0) (type default))
+  )
+  (wire (pts (xy 147.955 32.385) (xy 147.955 21.59))
+    (stroke (width 0) (type default))
+  )
+  (wire (pts (xy 142.24 32.385) (xy 142.24 15.24))
+    (stroke (width 0) (type default))
+  )
+  (wire (pts (xy 150.495 24.765) (xy 162.56 24.765))
+    (stroke (width 0) (type default))
+  )
+  (wire (pts (xy 44.45 19.685) (xy 55.245 19.685))
+    (stroke (width 0) (type default))
+  )
+  (wire (pts (xy 65.405 15.875) (xy 65.405 19.685))
+    (stroke (width 0) (type default))
+  )
+  (wire (pts (xy 144.78 18.415) (xy 162.56 18.415))
+    (stroke (width 0) (type default))
+  )
+  (wire (pts (xy 65.405 19.685) (xy 138.43 19.685))
+    (stroke (width 0) (type default))
+  )
+  (wire (pts (xy 142.24 15.24) (xy 162.56 15.24))
+    (stroke (width 0) (type default))
+  )
   (text "BANK_15\n" (at 46.99 139.065 0)
     (effects (font (size 5 5) (thickness 0.6) bold) (justify left bottom))
@@
     (effects (font (size 5 5) (thickness 0.6) bold) (justify left bottom))
   )
+  (label "TMS" (at 152.4 15.24 0) (fields_autoplaced)
+    (effects (font (size 1.27 1.27)) (justify left bottom))
+  )
+  (label "TDO_FPGA" (at 152.4 24.765 0) (fields_autoplaced)
+    (effects (font (size 1.27 1.27)) (justify left bottom))
+  )
+  (label "VCC1V8" (at 46.99 17.145 0) (fields_autoplaced)
+    (effects (font (size 1.27 1.27)) (justify left bottom))
+  )
+  (label "VCC3V3" (at 97.79 19.685 0) (fields_autoplaced)
+    (effects (font (size 1.27 1.27)) (justify left bottom))
+  )
+  (label "TCLK" (at 152.4 18.415 0) (fields_autoplaced)
+    (effects (font (size 1.27 1.27)) (justify left bottom))
+  )
+  (label "TDI_FPGA" (at 152.4 21.59 0) (fields_autoplaced)
+    (effects (font (size 1.27 1.27)) (justify left bottom))
+  )
+  (label "VCC1V0" (at 46.99 19.685 0) (fields_autoplaced)
+    (effects (font (size 1.27 1.27)) (justify left bottom))
+  )
+  (hierarchical_label "TCLK" (shape output) (at 162.56 18.415 0) (fields_autoplaced)
+    (effects (font (size 1.27 1.27)) (justify left))
+  )
+  (hierarchical_label "TDI_FPGA" (shape output) (at 162.56 21.59 0) (fields_autoplaced)
+    (effects (font (size 1.27 1.27)) (justify left))
+  )
+  (hierarchical_label "VCC1V0" (shape output) (at 44.45 19.685 180) (fields_autoplaced)
+    (effects (font (size 1.27 1.27)) (justify right))
+  )
+  (hierarchical_label "VCC1V8" (shape output) (at 44.45 17.145 180) (fields_autoplaced)
+    (effects (font (size 1.27 1.27)) (justify right))
+  )
+  (hierarchical_label "VCC3V3" (shape output) (at 68.58 15.875 0) (fields_autoplaced)
+    (effects (font (size 1.27 1.27)) (justify left))
+  )
+  (hierarchical_label "TDO_FPGA" (shape output) (at 162.56 24.765 0) (fields_autoplaced)
+    (effects (font (size 1.27 1.27)) (justify left))
+  )
+  (hierarchical_label "TMS" (shape output) (at 162.56 15.24 0) (fields_autoplaced)
+    (effects (font (size 1.27 1.27)) (justify left))
+  )
   (sheet (at 35.56 32.385) (size 53.975 60.325) (fields_autoplaced)
     (stroke (width 0.1524) (type solid))
@@
     (property "Field2" "" (at 35.56 32.385 0)
       (effects (font (size 1.27 1.27)) hide)
+    )
+    (pin "VCC1V0" output (at 55.245 32.385 90)
+      (effects (font (size 1.27 1.27)) (justify right))
+    )
+    (pin "VCC1V8" output (at 60.325 32.385 90)
+      (effects (font (size 1.27 1.27)) (justify right))
+    )
+    (pin "VCC3V3" output (at 65.405 32.385 90)
+      (effects (font (size 1.27 1.27)) (justify right))
     )
     (instances
@@
       (effects (font (size 1.27 1.27)) hide)
     )
+    (pin "VCC3V3" input (at 138.43 32.385 90)
+      (effects (font (size 1.27 1.27)) (justify right))
+    )
+    (pin "TMS" input (at 142.24 32.385 90)
+      (effects (font (size 1.27 1.27)) (justify right))
+    )
+    (pin "TCLK" input (at 144.78 32.385 90)
+      (effects (font (size 1.27 1.27)) (justify right))
+    )
+    (pin "TDI_FPGA" input (at 147.955 32.385 90)
+      (effects (font (size 1.27 1.27)) (justify right))
+    )
+    (pin "TDO_FPGA" input (at 150.495 32.385 90)
+      (effects (font (size 1.27 1.27)) (justify right))
+    )
     (instances

Commit message: updated schematic
Parts:
- added R29 (x4): 0, Resistor_SMD:R_0402_1005Metric_Pad0.72x0.64mm_HandSolder, symbol Device:R_Small_US
Connections:
- new net BANK_14/RXD_OUT: R29.1, R29.1
- new net BANK_14/TXD_IN: R29.1, R29.1
- new net RXD: R29.2, R29.2
- new net TXD: R29.2, R29.2
Other:
- sheet BANK_14 ports: added RXD_OUT, TXD_IN; removed none

Commit message: pcb layout updated
Parts:
- added J2: Conn_02x10_Odd_Even, Connector_PinHeader_1.27mm:PinHeader_2x10_P1.27mm_Vertical_SMD, symbol Connector_Generic:Conn_02x10_Odd_Even
- added J3: Conn_02x05_Odd_Even, Connector_PinHeader_1.27mm:PinHeader_2x05_P1.27mm_Vertical_SMD, symbol Connector_Generic:Conn_02x05_Odd_Even
- added J4: Conn_02x06_Odd_Even, Connector_PinHeader_1.27mm:PinHeader_2x06_P1.27mm_Vertical_SMD, symbol Connector_Generic:Conn_02x06_Odd_Even
Connections:
- new net BANK_14/PIO16: J2.2 (Pin_2)
- new net BANK_14/PIO17: J2.4 (Pin_4)
- new net BANK_14/PIO18: J2.6 (Pin_6)
- new net BANK_14/PIO19: J2.8 (Pin_8)
- new net BANK_14/PIO20: J2.10 (Pin_10)
- new net BANK_14/PIO21: J2.12 (Pin_12)
- new net BANK_14/PIO22: J2.14 (Pin_14)
- new net BANK_14/PIO23: J2.16 (Pin_16)
- new net BANK_14/PIO26: J2.18 (Pin_18)
- new net BANK_14/PIO27: J2.20 (Pin_20)
- new net BANK_14/PIO28: J2.19 (Pin_19)
- new net BANK_14/PIO29: J4.2 (Pin_2)
- new net BANK_14/PIO30: J4.4 (Pin_4)
- new net BANK_14/PIO31: J4.6 (Pin_6)
- new net BANK_15/AIN32: J3.3 (Pin_3)
- new net BANK_15/AIN33: J3.1 (Pin_1)
- new net BANK_34/JA1: J3.2 (Pin_2)
- new net BANK_34/JA10: J3.5 (Pin_5)
- new net BANK_34/JA2: J3.4 (Pin_4)
- new net BANK_34/JA3: J3.6 (Pin_6)
- new net BANK_34/JA4: J3.8 (Pin_8)
- new net BANK_34/JA7: J3.10 (Pin_10)
- new net BANK_34/JA8: J3.9 (Pin_9)
- new net BANK_34/JA9: J3.7 (Pin_7)
- new net BANK_34/PIO01: J2.1 (Pin_1)
- new net BANK_34/PIO02: J2.3 (Pin_3)
- new net BANK_34/PIO03: J2.5 (Pin_5)
- new net BANK_34/PIO04: J2.7 (Pin_7)
- new net BANK_34/PIO05: J2.9 (Pin_9)
- new net BANK_34/PIO06: J2.11 (Pin_11)
- new net BANK_34/PIO07: J2.13 (Pin_13)
- new net BANK_34/PIO08: J2.15 (Pin_15)
- new net BANK_34/PIO09: J2.17 (Pin_17)
- new net BANK_34/PIO40: J4.1 (Pin_1)
- new net BANK_34/PIO41: J4.3 (Pin_3)
- new net BANK_34/PIO42: J4.5 (Pin_5)
- new net BANK_34/PIO43: J4.7 (Pin_7)
- new net BANK_34/PIO44: J4.9 (Pin_9)
- new net BANK_34/PIO45: J4.11 (Pin_11)
- new net BANK_34/PIO46: J4.12 (Pin_12)
- new net BANK_34/PIO47: J4.10 (Pin_10)
- new net BANK_34/PIO48: J4.8 (Pin_8)
Other:
- sheet BANK_14 ports: added PIO16, PIO17, PIO18, PIO19, PIO20, PIO21, PIO22, PIO23, PIO26, PIO27, PIO28, PIO29, PIO30, PIO31; removed none
- sheet BANK_15 ports: added AIN32, AIN33; removed none
- sheet BANK_34 ports: added JA1, JA10, JA2, JA3, JA4, JA7, JA8, JA9, PIO01, PIO02, PIO03, PIO04, PIO05, PIO06, PIO07, PIO08, PIO09, PIO40, PIO41, PIO42, PIO43, PIO44, PIO45, PIO46, PIO47, PIO48; removed none
- moved on the sheet: R29

Commit message: updated files
Connections:
- net BANK_15/AIN32: now also J3.8 (Pin_8); no longer J3.3 (Pin_3)
- net BANK_15/AIN33: now also J3.10 (Pin_10); no longer J3.1 (Pin_1)
- net BANK_34/JA1: now also J3.9 (Pin_9); no longer J3.2 (Pin_2)
- net BANK_34/JA10: now also J3.6 (Pin_6); no longer J3.5 (Pin_5)
- net BANK_34/JA2: now also J3.7 (Pin_7); no longer J3.4 (Pin_4)
- net BANK_34/JA3: now also J3.5 (Pin_5); no longer J3.6 (Pin_6)
- net BANK_34/JA4: now also J3.3 (Pin_3); no longer J3.8 (Pin_8)
- net BANK_34/JA7: now also J3.1 (Pin_1); no longer J3.10 (Pin_10)
- net BANK_34/JA8: now also J3.2 (Pin_2); no longer J3.9 (Pin_9)
- net BANK_34/JA9: now also J3.4 (Pin_4); no longer J3.7 (Pin_7)
Other:
- moved on the sheet: J3
