File: kicad_files/FTDI.kicad_sch (KiCad schematic)
At the start: 1 part, among them IC2 FT2232HQ-TRAY

Commit message: schematic updated
Parts:
- removed IC2: FT2232HQ-TRAY, QFN50P900X900X90-65N-D, symbol SamacSys_Parts:FT2232HQ-TRAY
- added C53, C54: 12pf, Capacitor_SMD:C_0402_1005Metric_Pad0.74x0.62mm_HandSolder, symbol Device:C_Small
- added C55, C56, C57, C69: 4.7uf, Capacitor_SMD:C_0402_1005Metric_Pad0.74x0.62mm_HandSolder, symbol Device:C_Small
- added C58, C59, C60, C61, C62, C63, C64, C65, C67, C68, C70: 100nf, Capacitor_SMD:C_0402_1005Metric_Pad0.74x0.62mm_HandSolder, symbol Device:C_Small
- added C66: 1uf, Capacitor_SMD:C_0402_1005Metric_Pad0.74x0.62mm_HandSolder, symbol Device:C_Small
- added D3: LRB520G-30T1G, SamacSys_Parts:BZX84B2V7215, symbol Device:D_Schottky_Small
- added D5, D6: LED_Small, LED_SMD:LED_0402_1005Metric_Pad0.77x0.64mm_HandSolder, symbol Device:LED_Small
- added IC4: 74AHCT125BQ-Q100,1, SamacSys_Parts:74AHCT125BQQ1001, symbol SamacSys_Parts:74AHCT125BQ-Q100,1
- added IC5: M74VHC1GT04DTT1G, SamacSys_Parts:SOT95P275X110-5N, symbol SamacSys_Parts:M74VHC1GT04DTT1G
- added L4, L5: 1K 100MHz, symbol Device:L_Small
- added R29 (x3): 33, Resistor_SMD:R_0402_1005Metric_Pad0.72x0.64mm_HandSolder, symbol Device:R_Small_US
- added R29: 12K, Resistor_SMD:R_0402_1005Metric_Pad0.72x0.64mm_HandSolder, symbol Device:R_Small_US
- added R29: 1K, Resistor_SMD:R_0402_1005Metric_Pad0.72x0.64mm_HandSolder, symbol Device:R_Small_US
- added R43, R44: 2.2K, Resistor_SMD:R_0402_1005Metric_Pad0.72x0.64mm_HandSolder, symbol Device:R_Small_US
- added R45: 10K, Resistor_SMD:R_0402_1005Metric_Pad0.72x0.64mm_HandSolder, symbol Device:R_Small_US
- added U2: FT2232HQ, Package_DFN_QFN:QFN-64-1EP_9x9mm_P0.5mm_EP4.35x4.35mm, symbol Interface_USB:FT2232HQ
- added Y1: ABM3B-12.000MHZ-12-N2Y-T, SamacSys_Parts:ABM3B, symbol SamacSys_Parts:ABM3B-12.000MHZ-12-N2Y-T
Connections:
- new net: D6.2 (A), R44.1
- new net: C54.1, U2.2 (OSCI), Y1.1 (XTAL_1)
- new net: C53.1, U2.3 (OSCO), Y1.3 (XTAL_2)
- new net: C56.1, U2.50 (VREGIN)
- new net: R29.2, U2.61 (EEDATA)
- new net: R29.2, U2.62 (EECLK)
- new net: R29.2, U2.63 (EECS)
- new net: D3.2 (A), IC5.4 (OUT_~{Y}), R45.1
- new net: D5.2 (A), R43.1
- new net +1V8: C55.1, C58.1, C59.1, C60.1, U2.12 (VCORE), U2.37 (VCORE), U2.49 (VREGOUT), U2.64 (VCORE)
- new net +3V3: C61.1, C62.1, C63.1, C64.1, C65.1, C67.1, IC4.14 (VCC), IC5.5 (VCC), L4.1, L5.1, R43.2, R44.2, U2.20 (VCCIO), U2.31 (VCCIO), U2.42 (VCCIO), U2.56 (VCCIO)
- new net EECLK: R29.1
- new net EECS: R29.1
- new net EEDATA: R29.1
- new net ESP_EN: IC5.2 (INA)
- new net ESP_EN_N: C66.1, D3.1 (K), IC4.1 (1~{OE}), IC4.10 (3~{OE}), IC4.13 (4~{OE}), IC4.4 (2~{OE}), R45.2
- new net FT_RXD: U2.39 (BDBUS1)
- new net FT_TCK: IC4.12 (4A), U2.16 (ADBUS0)
- new net FT_TDI: IC4.9 (3A), U2.17 (ADBUS1)
- new net FT_TDO: IC4.5 (2A), U2.18 (ADBUS2)
- new net FT_TMS: IC4.2 (1A), U2.19 (ADBUS3)
- new net FT_TXD: U2.38 (BDBUS0)
- new net FT_nDTR: U2.43 (BDBUS4)
- new net FT_nRTS: U2.40 (BDBUS2)
- new net FT_nRXLED: D5.1 (K), U2.54 (BCBUS3)
- new net FT_nTXLED: D6.1 (K), U2.55 (BCBUS4)
- new net GND: C53.2, C54.2, C55.2, C56.2, C57.2, C58.2, C59.2, C60.2, C61.2, C62.2, C63.2, C64.2, C65.2, C66.2, C67.2, C68.2, C69.2, C70.2, IC4.15 (GND_2), IC4.7 (GND_1), IC5.3 (GND), R29.1, U2.1 (GND), U2.10 (AGND), U2.11 (GND), U2.13 (TEST), U2.15 (GND), U2.25 (GND), U2.35 (GND), U2.47 (GND), U2.5 (GND), U2.51 (GND), U2.65 (GND), Y1.2 (GND_1), Y1.4 (GND_2)
- new net REF: R29.2, U2.6 (REF)
- new net RESET: R29.2, U2.14 (~{RESET})
- new net TCK: IC4.11 (4Y)
- new net TDI: IC4.8 (3Y)
- new net TDO: IC4.6 (2Y)
- new net TMS: IC4.3 (1Y)
- new net USB_DM: U2.7 (DM)
- new net USB_DP: U2.8 (DP)
- new net VDD3V3: R29.1
- new net VPHY: C57.1, C68.1, L4.2, U2.4 (VPHY)
- new net VPLL: C69.1, C70.1, L5.2, U2.9 (VPLL)
- no-connect marks 0 -> 24

Commit message: updated schematic
Parts:
- added C71: 10uf, Capacitor_SMD:C_0603_1608Metric, symbol Device:C_Small
- added D10, D11, D8: LESD5D5.0CT1G, SamacSys_Parts:LESD5D50CT1G, symbol Device:D_TVS_Filled
- added J1: U254-051N-4BH806, footprints:U254-051N-4BH806, symbol KiCadSymbols:USB_B_10118193-0001LF
- added R29 (x4): 0, Resistor_SMD:R_0402_1005Metric_Pad0.72x0.64mm_HandSolder, symbol Device:R_Small_US
Connections:
- net +3V3: now also C56.1, U2.50 (VREGIN)
- net FT_RXD: now also R29.1
- net FT_TXD: now also R29.1
- net GND: now also C71.2, D10.1 (A1), D11.1 (A1), D8.1 (A1), J1.5 (GND), J1.6 (S1), J1.7 (S2), J1.8 (S3), J1.9 (S4)
- net USB_DM: now also R29.2
- net USB_DP: now also R29.2
- new net: D10.2 (A2), J1.2 (D-), R29.1
- new net: D11.2 (A2), J1.3 (D+), R29.1
- new net RXD: R29.2
- new net TXD: R29.2
- new net USB5V0: C71.1, D8.2 (A2), J1.1 (VUSB)
- no-connect marks 24 -> 25
Other:
- note added: "Decoupling Caps"
- note added: "Inverters"
- moved on the sheet: C53, C54, C55, C56, C57, C58, C59, C60, C61, C62, C63, C64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

Commit message: BGA Routing started
Parts:
- added C74: 100nf, Capacitor_SMD:C_0402_1005Metric_Pad0.74x0.62mm_HandSolder, symbol Device:C_Small
- added IC6: M93C46-WMN6TP, SOIC127P600X175-8N, symbol SamacSys_Parts:M93C46-WMN6TP
- added R29 (x2): 0, Resistor_SMD:R_0402_1005Metric_Pad0.72x0.64mm_HandSolder, symbol Device:R_Small_US
- added R29 (x3): 10K, Resistor_SMD:R_0402_1005Metric_Pad0.72x0.64mm_HandSolder, symbol Device:R_Small_US
- added R29: 2.2K, Resistor_SMD:R_0402_1005Metric_Pad0.72x0.64mm_HandSolder, symbol Device:R_Small_US
- IC4: footprint SamacSys_Parts:74AHCT125BQQ1001 -> SamacSys_Parts:SOIC127P600X175-14N
- L4, L5: footprint (none) -> Inductor_SMD:L_0402_1005Metric_Pad0.77x0.64mm_HandSolder
Connections:
- net +3V3: now also C74.1, IC6.8 (VCC), R29.2, R29.2, R29.2, R29.2
- net EECLK: now also IC6.2 (C), R29.1
- net EECS: now also IC6.1 (S), R29.1
- net EEDATA: now also IC6.3 (D), R29.1
- net GND: now also C74.2, IC6.5 (VSS), R29.2
- net USB_DM renamed USB_D-
- net USB_DP renamed USB_D+
- new net: IC6.4 (Q), R29.1, R29.2
- new net: IC6.6 (ORG), R29.1
- new net: IC6.7 (DU), R29.1

Commit message: pcb layout updated
Parts:
- IC6: footprint SOIC127P600X175-8N -> SamacSys_Parts:SOIC127P600X175-8N
Connections:
- net GND: no longer IC4.15 (GND_2)
Other:
- moved on the sheet: C65
Changed lines of the file:
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@@
   (junction (at 68.58 71.755) (diameter 0) (color 0 0 0 0)
   )
+  (junction (at 382.27 104.775) (diameter 0) (color 0 0 0 0)
+  )
   (junction (at 159.385 55.245) (diameter 0) (color 0 0 0 0)
   )
@@
   (junction (at 48.26 144.145) (diameter 0) (color 0 0 0 0)
   )
-  (junction (at 359.41 101.6) (diameter 0) (color 0 0 0 0)
+  (junction (at 359.41 95.885) (diameter 0) (color 0 0 0 0)
   )
   (junction (at 168.91 55.245) (diameter 0) (color 0 0 0 0)
@@
   (junction (at 176.53 215.265) (diameter 0) (color 0 0 0 0)
   )
-  (junction (at 378.46 94.615) (diameter 0) (color 0 0 0 0)
-  )
-  (junction (at 378.46 99.695) (diameter 0) (color 0 0 0 0)
-  )
   (junction (at 89.535 128.905) (diameter 0) (color 0 0 0 0)
   )
@@
   (junction (at 222.25 215.265) (diameter 0) (color 0 0 0 0)
   )
-  (junction (at 359.41 102.87) (diameter 0) (color 0 0 0 0)
+  (junction (at 359.41 97.155) (diameter 0) (color 0 0 0 0)
   )
-  (junction (at 359.41 100.33) (diameter 0) (color 0 0 0 0)
+  (junction (at 359.41 94.615) (diameter 0) (color 0 0 0 0)
   )
   (junction (at 57.15 128.905) (diameter 0) (color 0 0 0 0)
@@
     (stroke (width 0) (type default))
   )
-  (wire (pts (xy 382.27 87.63) (xy 382.27 91.44))
+  (wire (pts (xy 382.27 87.63) (xy 382.27 93.345))
     (stroke (width 0) (type default))
   )
@@
     (stroke (width 0) (type default))
   )
-  (wire (pts (xy 378.46 99.695) (xy 378.46 101.6))
-    (stroke (width 0) (type default))
-  )
   (wire (pts (xy 44.45 133.985) (xy 79.375 133.985))
     (stroke (width 0) (type default))
@@
     (stroke (width 0) (type default))
   )
-  (wire (pts (xy 349.885 92.075) (xy 378.46 92.075))
-    (stroke (width 0) (type default))
-  )
   (wire (pts (xy 89.535 147.955) (xy 89.535 159.385))
     (stroke (width 0) (type default))
   )
-  (wire (pts (xy 382.27 96.52) (xy 382.27 99.695))
+  (wire (pts (xy 382.27 98.425) (xy 382.27 104.775))
     (stroke (width 0) (type default))
   )
@@
     (stroke (width 0) (type default))
   )
-  (wire (pts (xy 359.41 102.87) (xy 359.41 105.41))
+  (wire (pts (xy 359.41 97.155) (xy 359.41 99.695))
     (stroke (width 0) (type default))
   )
@@
     (stroke (width 0) (type default))
   )
-  (wire (pts (xy 378.46 92.075) (xy 378.46 94.615))
-    (stroke (width 0) (type default))
-  )
   (wire (pts (xy 168.275 189.865) (xy 172.085 189.865))
     (stroke (width 0) (type default))
@@
     (stroke (width 0) (type default))
   )
-  (wire (pts (xy 378.46 94.615) (xy 378.46 99.695))
-    (stroke (width 0) (type default))
-  )
   (wire (pts (xy 234.95 83.185) (xy 234.95 90.805))
     (stroke (width 0) (type default))
@@
     (stroke (width 0) (type default))
   )
+  (wire (pts (xy 349.885 104.775) (xy 382.27 104.775))
+    (stroke (width 0) (type default))
+  )
   (wire (pts (xy 172.085 215.265) (xy 176.53 215.265))
     (stroke (width 0) (type default))
@@
     (stroke (width 0) (type default))
   )
-  (wire (pts (xy 359.41 101.6) (xy 372.11 101.6))
+  (wire (pts (xy 359.41 95.885) (xy 372.11 95.885))
     (stroke (width 0) (type default))
   )
@@
     (stroke (width 0) (type default))
   )
-  (wire (pts (xy 359.41 101.6) (xy 359.41 102.87))
+  (wire (pts (xy 359.41 95.885) (xy 359.41 97.155))
     (stroke (width 0) (type default))
   )
@@
     (stroke (width 0) (type default))
   )
-  (wire (pts (xy 378.46 99.695) (xy 382.27 99.695))
-    (stroke (width 0) (type default))
-  )
   (polyline (pts (xy 17.78 104.775) (xy 90.805 104.775))
     (stroke (width 0) (type default))
@@
     (stroke (width 0) (type default))
   )
-  (wire (pts (xy 359.41 105.41) (xy 349.885 105.41))
+  (wire (pts (xy 359.41 99.695) (xy 349.885 99.695))
     (stroke (width 0) (type default))
   )
@@
     (stroke (width 0) (type default))
   )
-  (wire (pts (xy 359.41 97.79) (xy 359.41 100.33))
+  (wire (pts (xy 359.41 92.075) (xy 359.41 94.615))
     (stroke (width 0) (type default))
   )
@@
     (stroke (width 0) (type default))
   )
-  (wire (pts (xy 349.885 94.615) (xy 378.46 94.615))
-    (stroke (width 0) (type default))
-  )
   (wire (pts (xy 167.005 98.425) (xy 167.005 104.775))
     (stroke (width 0) (type default))
@@
     (stroke (width 0) (type default))
   )
-  (wire (pts (xy 359.41 102.87) (xy 349.885 102.87))
+  (wire (pts (xy 359.41 97.155) (xy 349.885 97.155))
     (stroke (width 0) (type default))
   )
@@
     (stroke (width 0) (type default))
   )
-  (wire (pts (xy 359.41 100.33) (xy 349.885 100.33))
+  (wire (pts (xy 359.41 94.615) (xy 349.885 94.615))
     (stroke (width 0) (type default))
   )
@@
     (stroke (width 0) (type default))
   )
-  (wire (pts (xy 359.41 100.33) (xy 359.41 101.6))
+  (wire (pts (xy 359.41 94.615) (xy 359.41 95.885))
     (stroke (width 0) (type default))
   )
@@
     (stroke (width 0) (type default))
   )
-  (wire (pts (xy 359.41 97.79) (xy 349.885 97.79))
+  (wire (pts (xy 359.41 92.075) (xy 349.885 92.075))
     (stroke (width 0) (type default))
   )
@@
     (stroke (width 0) (type default))
   )
+  (wire (pts (xy 382.27 107.95) (xy 382.27 104.775))
+    (stroke (width 0) (type default))
+  )
   (wire (pts (xy 300.99 174.625) (xy 300.99 177.165))
     (stroke (width 0) (type default))
@@
     (effects (font (size 1.27 1.27)) (justify right bottom))
   )
-  (label "ESP_EN_N" (at 372.11 101.6 180) (fields_autoplaced)
+  (label "ESP_EN_N" (at 372.11 95.885 180) (fields_autoplaced)
     (effects (font (size 1.27 1.27)) (justify right bottom))
   )
@@
       (effects (font (size 1.27 1.27)))
     )
-    (property "Footprint" "SOIC127P600X175-8N" (at 83.82 296.85 0)
+    (property "Footprint" "SamacSys_Parts:SOIC127P600X175-8N" (at 83.82 296.85 0)
       (effects (font (size 1.27 1.27)) (justify left top) hide)
     )
@@
     (pin "13")
     (pin "14")
-    (pin "15")
     (pin "2")
     (pin "3")
@@
     )
   )
-  (symbol (lib_id "Device:C_Small") (at 382.27 93.98 0) (unit 1)
+  (symbol (lib_id "Device:C_Small") (at 382.27 95.885 0) (unit 1)
     (in_bom yes) (on_board yes) (dnp no) (fields_autoplaced)
-    (property "Reference" "C65" (at 384.81 93.3513 0)
+    (property "Reference" "C65" (at 384.81 95.2563 0)
       (effects (font (size 1.27 1.27)) (justify left))
     )
-    (property "Value" "100nf" (at 384.81 95.8913 0)
+    (property "Value" "100nf" (at 384.81 97.7963 0)
       (effects (font (size 1.27 1.27)) (justify left))
     )
-    (property "Footprint" "Capacitor_SMD:C_0402_1005Metric_Pad0.74x0.62mm_HandSolder" (at 382.27 93.98 0)
+    (property "Footprint" "Capacitor_SMD:C_0402_1005Metric_Pad0.74x0.62mm_HandSolder" (at 382.27 95.885 0)
       (effects (font (size 1.27 1.27)) hide)
     )
-    (property "Datasheet" "~" (at 382.27 93.98 0)
+    (property "Datasheet" "~" (at 382.27 95.885 0)
       (effects (font (size 1.27 1.27)) hide)
     )
@@
     )
   )
-  (symbol (lib_id "power:GND") (at 378.46 101.6 0) (unit 1)
+  (symbol (lib_id "power:GND") (at 382.27 107.95 0) (unit 1)
     (in_bom yes) (on_board yes) (dnp no)
-    (property "Reference" "#PWR010" (at 378.46 107.95 0)
+    (property "Reference" "#PWR010" (at 382.27 114.3 0)
       (effects (font (size 1.27 1.27)) hide)
     )
-    (property "Value" "GND" (at 378.46 105.41 0)
+    (property "Value" "GND" (at 382.27 111.76 0)
       (effects (font (size 1.27 1.27)))
     )
-    (property "Footprint" "" (at 378.46 101.6 0)
+    (property "Footprint" "" (at 382.27 107.95 0)
       (effects (font (size 1.27 1.27)) hide)
     )
-    (property "Datasheet" "" (at 378.46 101.6 0)
+    (property "Datasheet" "" (at 382.27 107.95 0)
       (effects (font (size 1.27 1.27)) hide)
     )

Commit message: updated layout
Parts:
- L4, L5: footprint Inductor_SMD:L_0402_1005Metric_Pad0.77x0.64mm_HandSolder -> Inductor_SMD:L_0603_1608Metric_Pad1.05x0.95mm_HandSolder
Changed lines of the file:
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@@
       (effects (font (size 1.27 1.27)))
     )
-    (property "Footprint" "Inductor_SMD:L_0402_1005Metric_Pad0.77x0.64mm_HandSolder" (at 49.53 71.755 0)
+    (property "Footprint" "Inductor_SMD:L_0603_1608Metric_Pad1.05x0.95mm_HandSolder" (at 49.53 71.755 0)
       (effects (font (size 1.27 1.27)) hide)
     )
@@
       (effects (font (size 1.27 1.27)))
     )
-    (property "Footprint" "Inductor_SMD:L_0402_1005Metric_Pad0.77x0.64mm_HandSolder" (at 49.53 40.005 0)
+    (property "Footprint" "Inductor_SMD:L_0603_1608Metric_Pad1.05x0.95mm_HandSolder" (at 49.53 40.005 0)
       (effects (font (size 1.27 1.27)) hide)
     )

Commit message: layout basic completed
Connections:
- net VDD3V3 is gone; now on net +3V3: R29.1
Changed lines of the file:
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@@
+    (effects (font (size 1.27 1.27)) (justify left bottom))
+  )
+  (label "VDD3V3" (at 152.4 37.465 0) (fields_autoplaced)
     (effects (font (size 1.27 1.27)) (justify left bottom))
   )

Commit message: updated files
Other:
- note added: "EEPROM"
- note added: "External Nets"
- note added: "FTDI_Chips"
- note added: "USB Connectors"
- moved on the sheet: C74, IC6, R29
