File: kicad_files/sparton_7.kicad_sch (KiCad schematic)
At the start: 1 part, among them IC1 XC7S25-1CSGA225C

Commit message: working
Other:
- moved on the sheet: IC1A

Commit message: schematic updated
Parts:
- removed IC1: XC7S25-1CSGA225C, BGA225C80P15X15_1300X1300X140, symbol SamacSys_Parts:XC7S25-1CSGA225C
Other:
- added sheet FPGA_SPARTAN_7 (FPGA_SPARTAN_7.kicad_sch)
- note added: "SPARTAN_7"

Commit message: ftdi progess
Other:
- added sheet FTDI (FTDI.kicad_sch)
- note added: "FTDI2232H"
Changed lines of the file:
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@@
 (kicad_sch (version 20230121) (generator eeschema)
   (paper "A3")
+  (text "FTDI2232H\n" (at 66.675 156.845 0)
+    (effects (font (size 5 5) (thickness 0.6) bold) (justify left bottom))
+  )
   (text "SPARTAN_7\n" (at 176.53 156.845 0)
     (effects (font (size 5 5) (thickness 0.6) bold) (justify left bottom))
@@
       )
     )
+  )
+  (sheet (at 45.72 109.855) (size 79.375 93.345) (fields_autoplaced)
+    (stroke (width 0.1524) (type solid))
+    (fill (color 0 0 0 0.0000))
+    (property "Sheetname" "FTDI" (at 45.72 109.1434 0)
+      (effects (font (size 1.27 1.27)) (justify left bottom))
+    )
+    (property "Sheetfile" "FTDI.kicad_sch" (at 45.72 203.7846 0)
+      (effects (font (size 1.27 1.27)) (justify left top))
+    )
+    (property "Field2" "" (at 45.72 109.855 0)
+      (effects (font (size 1.27 1.27)) hide)
+    )
+    (property "Field3" "" (at 45.72 109.855 0)
+      (effects (font (size 1.27 1.27)) hide)
+    )
+    (instances
+      (project "sparton_7"
+        (path "/94bd3a84-5526-4cf2-a5cc-3887356f447c" (page "8"))
+      )
+    )

Commit message: schematic updated
Other:
- added sheet POWER_REGULATOR (POWER_REGULATOR.kicad_sch)
- sheet FPGA_SPARTAN_7 ports: added TCLK, TDI_FPGA, TDO_FPGA, TMS, VCC1V0, VCC1V8, VCC3V3; removed none
- sheet FTDI ports: added TCK, TDI, TDO, TMS; removed none
- note added: "POWER_REGULATOR"
Changed lines of the file:
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@@
 (kicad_sch (version 20230121) (generator eeschema)
   (paper "A3")
+  (wire (pts (xy 125.095 139.065) (xy 150.495 139.065))
+    (stroke (width 0) (type default))
+  )
+  (wire (pts (xy 139.7 102.235) (xy 199.39 102.235))
+    (stroke (width 0) (type default))
+  )
+  (wire (pts (xy 135.89 89.535) (xy 135.89 105.41))
+    (stroke (width 0) (type default))
+  )
+  (wire (pts (xy 139.7 89.535) (xy 139.7 102.235))
+    (stroke (width 0) (type default))
+  )
+  (wire (pts (xy 125.095 144.145) (xy 150.495 144.145))
+    (stroke (width 0) (type default))
+  )
+  (wire (pts (xy 135.89 105.41) (xy 196.215 105.41))
+    (stroke (width 0) (type default))
+  )
+  (wire (pts (xy 199.39 102.235) (xy 199.39 112.395))
+    (stroke (width 0) (type default))
+  )
+  (wire (pts (xy 142.875 99.06) (xy 203.2 99.06))
+    (stroke (width 0) (type default))
+  )
+  (wire (pts (xy 203.2 99.06) (xy 203.2 112.395))
+    (stroke (width 0) (type default))
+  )
+  (wire (pts (xy 196.215 105.41) (xy 196.215 112.395))
+    (stroke (width 0) (type default))
+  )
+  (wire (pts (xy 125.095 136.525) (xy 150.495 136.525))
+    (stroke (width 0) (type default))
+  )
+  (wire (pts (xy 125.095 141.605) (xy 150.495 141.605))
+    (stroke (width 0) (type default))
+  )
+  (wire (pts (xy 142.875 89.535) (xy 142.875 99.06))
+    (stroke (width 0) (type default))
+  )
   (text "FTDI2232H\n" (at 66.675 156.845 0)
     (effects (font (size 5 5) (thickness 0.6) bold) (justify left bottom))
@@
     (effects (font (size 5 5) (thickness 0.6) bold) (justify left bottom))
   )
-  (sheet (at 149.225 110.49) (size 101.6 93.345) (fields_autoplaced)
+  (text "POWER_REGULATOR\n" (at 104.14 64.135 0)
+    (effects (font (size 5 5) (thickness 0.6) bold) (justify left bottom))
+  )
+  (sheet (at 67.945 35.56) (size 139.065 53.975) (fields_autoplaced)
     (stroke (width 0.1524) (type solid))
     (fill (color 0 0 0 0.0000))
-    (property "Sheetname" "FPGA_SPARTAN_7" (at 149.225 109.7784 0)
+    (property "Sheetname" "POWER_REGULATOR" (at 67.945 34.8484 0)
       (effects (font (size 1.27 1.27)) (justify left bottom))
     )
-    (property "Sheetfile" "FPGA_SPARTAN_7.kicad_sch" (at 149.225 204.4196 0)
+    (property "Sheetfile" "POWER_REGULATOR.kicad_sch" (at 67.945 90.1196 0)
       (effects (font (size 1.27 1.27)) (justify left top))
+    )
+    (property "Field2" "" (at 67.945 35.56 0)
+      (effects (font (size 1.27 1.27)) hide)
+    )
+    (pin "VCC1V0" output (at 142.875 89.535 270)
+      (effects (font (size 1.27 1.27)) (justify left))
+    )
+    (pin "VCC1V8" output (at 139.7 89.535 270)
+      (effects (font (size 1.27 1.27)) (justify left))
+    )
+    (pin "VCC3V3" output (at 135.89 89.535 270)
+      (effects (font (size 1.27 1.27)) (justify left))
+    )
+    (instances
+      (project "sparton_7"
+        (path "/94bd3a84-5526-4cf2-a5cc-3887356f447c" (page "9"))
+      )
+    )
+  )
+  (sheet (at 150.495 112.395) (size 101.6 93.345) (fields_autoplaced)
+    (stroke (width 0.1524) (type solid))
+    (fill (color 0 0 0 0.0000))
+    (property "Sheetname" "FPGA_SPARTAN_7" (at 150.495 111.6834 0)
+      (effects (font (size 1.27 1.27)) (justify left bottom))
+    )
+    (property "Sheetfile" "FPGA_SPARTAN_7.kicad_sch" (at 150.495 206.3246 0)
+      (effects (font (size 1.27 1.27)) (justify left top))
+    )
+    (pin "TDI_FPGA" input (at 150.495 141.605 180)
+      (effects (font (size 1.27 1.27)) (justify left))
+    )
+    (pin "TMS" input (at 150.495 139.065 180)
+      (effects (font (size 1.27 1.27)) (justify left))
+    )
+    (pin "TCLK" input (at 150.495 136.525 180)
+      (effects (font (size 1.27 1.27)) (justify left))
+    )
+    (pin "TDO_FPGA" input (at 150.495 144.145 180)
+      (effects (font (size 1.27 1.27)) (justify left))
+    )
+    (pin "VCC1V8" output (at 199.39 112.395 90)
+      (effects (font (size 1.27 1.27)) (justify right))
+    )
+    (pin "VCC1V0" output (at 203.2 112.395 90)
+      (effects (font (size 1.27 1.27)) (justify right))
+    )
+    (pin "VCC3V3" output (at 196.215 112.395 90)
+      (effects (font (size 1.27 1.27)) (justify right))
     )
     (instances
@@
       (effects (font (size 1.27 1.27)) hide)
     )
+    (pin "TMS" output (at 125.095 139.065 0)
+      (effects (font (size 1.27 1.27)) (justify right))
+    )
+    (pin "TDO" output (at 125.095 144.145 0)
+      (effects (font (size 1.27 1.27)) (justify right))
+    )
+    (pin "TDI" output (at 125.095 141.605 0)
+      (effects (font (size 1.27 1.27)) (justify right))
+    )
+    (pin "TCK" output (at 125.095 136.525 0)
+      (effects (font (size 1.27 1.27)) (justify right))
+    )
     (instances

Commit message: updated schematic
Other:
- sheet FPGA_SPARTAN_7 ports: added RXD, TXD; removed none
- sheet FTDI ports: added +3V3, RXD, TXD, USB5V0; removed none
- sheet POWER_REGULATOR ports: added USB5V0, VU; removed none
Changed lines of the file:
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@@
 (kicad_sch (version 20230121) (generator eeschema)
   (paper "A3")
-  (wire (pts (xy 125.095 139.065) (xy 150.495 139.065))
+  (junction (at 135.89 105.41) (diameter 0) (color 0 0 0 0)
+  )
+  (wire (pts (xy 125.095 146.685) (xy 150.495 146.685))
     (stroke (width 0) (type default))
   )
@@
     (stroke (width 0) (type default))
   )
+  (wire (pts (xy 78.74 102.235) (xy 78.74 109.855))
+    (stroke (width 0) (type default))
+  )
   (wire (pts (xy 139.7 89.535) (xy 139.7 102.235))
     (stroke (width 0) (type default))
   )
-  (wire (pts (xy 125.095 144.145) (xy 150.495 144.145))
+  (wire (pts (xy 125.095 177.8) (xy 150.495 177.8))
+    (stroke (width 0) (type default))
+  )
+  (wire (pts (xy 125.095 161.29) (xy 150.495 161.29))
     (stroke (width 0) (type default))
   )
@@
     (stroke (width 0) (type default))
   )
-  (wire (pts (xy 199.39 102.235) (xy 199.39 112.395))
+  (wire (pts (xy 199.39 102.235) (xy 199.39 109.855))
+    (stroke (width 0) (type default))
+  )
+  (wire (pts (xy 132.08 102.235) (xy 78.74 102.235))
+    (stroke (width 0) (type default))
+  )
+  (wire (pts (xy 135.89 105.41) (xy 85.09 105.41))
     (stroke (width 0) (type default))
   )
@@
     (stroke (width 0) (type default))
   )
-  (wire (pts (xy 203.2 99.06) (xy 203.2 112.395))
+  (wire (pts (xy 203.2 99.06) (xy 203.2 109.855))
     (stroke (width 0) (type default))
   )
-  (wire (pts (xy 196.215 105.41) (xy 196.215 112.395))
+  (wire (pts (xy 125.095 130.81) (xy 150.495 130.81))
     (stroke (width 0) (type default))
   )
-  (wire (pts (xy 125.095 136.525) (xy 150.495 136.525))
+  (wire (pts (xy 196.215 105.41) (xy 196.215 109.855))
     (stroke (width 0) (type default))
   )
-  (wire (pts (xy 125.095 141.605) (xy 150.495 141.605))
+  (wire (pts (xy 132.08 89.535) (xy 132.08 102.235))
+    (stroke (width 0) (type default))
+  )
+  (wire (pts (xy 85.09 105.41) (xy 85.09 109.855))
+    (stroke (width 0) (type default))
+  )
+  (wire (pts (xy 125.095 189.865) (xy 150.495 189.865))
     (stroke (width 0) (type default))
   )
   (wire (pts (xy 142.875 89.535) (xy 142.875 99.06))
+    (stroke (width 0) (type default))
+  )
+  (wire (pts (xy 125.095 121.285) (xy 150.495 121.285))
     (stroke (width 0) (type default))
   )
@@
       (effects (font (size 1.27 1.27)) (justify left))
     )
+    (pin "VU" output (at 207.01 45.085 0)
+      (effects (font (size 1.27 1.27)) (justify right))
+    )
+    (pin "USB5V0" output (at 132.08 89.535 270)
+      (effects (font (size 1.27 1.27)) (justify left))
+    )
     (instances
       (project "sparton_7"
@@
     )
   )
-  (sheet (at 150.495 112.395) (size 101.6 93.345) (fields_autoplaced)
+  (sheet (at 150.495 109.855) (size 101.6 93.345) (fields_autoplaced)
     (stroke (width 0.1524) (type solid))
     (fill (color 0 0 0 0.0000))
-    (property "Sheetname" "FPGA_SPARTAN_7" (at 150.495 111.6834 0)
+    (property "Sheetname" "FPGA_SPARTAN_7" (at 150.495 109.1434 0)
       (effects (font (size 1.27 1.27)) (justify left bottom))
     )
-    (property "Sheetfile" "FPGA_SPARTAN_7.kicad_sch" (at 150.495 206.3246 0)
+    (property "Sheetfile" "FPGA_SPARTAN_7.kicad_sch" (at 150.495 203.7846 0)
       (effects (font (size 1.27 1.27)) (justify left top))
     )
-    (pin "TDI_FPGA" input (at 150.495 141.605 180)
+    (pin "TDI_FPGA" input (at 150.495 161.29 180)
       (effects (font (size 1.27 1.27)) (justify left))
     )
-    (pin "TMS" input (at 150.495 139.065 180)
+    (pin "TMS" input (at 150.495 146.685 180)
       (effects (font (size 1.27 1.27)) (justify left))
     )
-    (pin "TCLK" input (at 150.495 136.525 180)
+    (pin "TCLK" input (at 150.495 130.81 180)
       (effects (font (size 1.27 1.27)) (justify left))
     )
-    (pin "TDO_FPGA" input (at 150.495 144.145 180)
+    (pin "TDO_FPGA" input (at 150.495 177.8 180)
       (effects (font (size 1.27 1.27)) (justify left))
     )
-    (pin "VCC1V8" output (at 199.39 112.395 90)
+    (pin "VCC1V8" output (at 199.39 109.855 90)
       (effects (font (size 1.27 1.27)) (justify right))
     )
-    (pin "VCC1V0" output (at 203.2 112.395 90)
+    (pin "VCC1V0" output (at 203.2 109.855 90)
       (effects (font (size 1.27 1.27)) (justify right))
     )
-    (pin "VCC3V3" output (at 196.215 112.395 90)
+    (pin "VCC3V3" output (at 196.215 109.855 90)
       (effects (font (size 1.27 1.27)) (justify right))
+    )
+    (pin "TXD" output (at 150.495 121.285 180)
+      (effects (font (size 1.27 1.27)) (justify left))
+    )
+    (pin "RXD" output (at 150.495 189.865 180)
+      (effects (font (size 1.27 1.27)) (justify left))
     )
     (instances
@@
       (effects (font (size 1.27 1.27)) hide)
     )
-    (pin "TMS" output (at 125.095 139.065 0)
+    (pin "TMS" output (at 125.095 146.685 0)
       (effects (font (size 1.27 1.27)) (justify right))
     )
-    (pin "TDO" output (at 125.095 144.145 0)
+    (pin "TDO" output (at 125.095 177.8 0)
       (effects (font (size 1.27 1.27)) (justify right))
     )
-    (pin "TDI" output (at 125.095 141.605 0)
+    (pin "TDI" output (at 125.095 161.29 0)
       (effects (font (size 1.27 1.27)) (justify right))
     )
-    (pin "TCK" output (at 125.095 136.525 0)
+    (pin "TCK" output (at 125.095 130.81 0)
       (effects (font (size 1.27 1.27)) (justify right))
     )
+    (pin "+3V3" input (at 85.09 109.855 90)
+      (effects (font (size 1.27 1.27)) (justify right))
+    )
+    (pin "USB5V0" output (at 78.74 109.855 90)
+      (effects (font (size 1.27 1.27)) (justify right))
+    )
+    (pin "TXD" output (at 125.095 121.285 0)
+      (effects (font (size 1.27 1.27)) (justify right))
+    )
+    (pin "RXD" output (at 125.095 189.865 0)
+      (effects (font (size 1.27 1.27)) (justify right))
+    )

Commit message: updated files
Other:
- sheet FTDI ports: added +1V8; removed none
Changed lines of the file:
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@@
   (junction (at 135.89 105.41) (diameter 0) (color 0 0 0 0)
+  )
+  (junction (at 139.7 102.235) (diameter 0) (color 0 0 0 0)
+  )
+  (wire (pts (xy 125.095 114.935) (xy 139.7 114.935))
+    (stroke (width 0) (type default))
   )
   (wire (pts (xy 125.095 146.685) (xy 150.495 146.685))
@@
   )
   (wire (pts (xy 85.09 105.41) (xy 85.09 109.855))
+    (stroke (width 0) (type default))
+  )
+  (wire (pts (xy 139.7 114.935) (xy 139.7 102.235))
     (stroke (width 0) (type default))
   )
@@
       (effects (font (size 1.27 1.27)) (justify right))
     )
+    (pin "+1V8" input (at 125.095 114.935 0)
+      (effects (font (size 1.27 1.27)) (justify right))
+    )
