File: kicad_files/2030_Audio_Board.kicad_pcb (KiCad board)
At the start: 2 copper layers, 50 x 50 mm, 19 parts, among them U1 TDA2030

Commit message: routing compledted
Parts:
- added J1: Conn_01x02_Pin, footprints:JST_B2B-PH-K-S(LF)(SN), F.Cu at (103.4, 107.3)
- C3, C5, C6: footprint Capacitor_SMD:C_0603_1608Metric_Pad1.08x0.95mm_HandSolder -> Capacitor_SMD:C_0805_2012Metric_Pad1.18x1.45mm_HandSolder
- R1, R2, R3, R4, R5: footprint Resistor_SMD:R_0603_1608Metric_Pad0.98x0.95mm_HandSolder -> Resistor_SMD:R_0805_2012Metric_Pad1.20x1.40mm_HandSolder
- R6: footprint Resistor_SMD:R_1206_3216Metric_Pad1.30x1.75mm_HandSolder -> Resistor_THT:R_Axial_DIN0204_L3.6mm_D1.6mm_P7.62mm_Horizontal
- moved R5 42.1 mm to (126.0, 102.2), turned to 180 degrees
- moved R4 38.7 mm to (146.1, 117.5)
- moved C1 35.8 mm to (119.8, 123.7), turned to 180 degrees
- moved C2 34.1 mm to (132.1, 123.7)
- moved LS1 30.6 mm to (145.3, 124.7), turned to -90 degrees
- moved C6 27.9 mm to (141.0, 120.6), turned to 90 degrees
- moved C5 24.2 mm to (136.0, 116.2)
- moved C4 21.7 mm to (143.0, 118.5), turned to -90 degrees
- moved R3 19.1 mm to (122.7, 120.4), turned to 90 degrees
- moved R2 18.7 mm to (126.1, 120.4), turned to -90 degrees
- moved C7 13.7 mm to (142.3, 142.0), turned to 90 degrees
- moved C3 9.10 mm to (116.2, 116.2)
- moved D1 9.09 mm to (123.2, 135.6), turned to -90 degrees
- moved R1 8.57 mm to (123.2, 131.4), turned to -90 degrees
- moved R6 6.72 mm to (129.5, 145.8), turned to 90 degrees
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Routing:
- net Net-(D1-A): track 0.00 -> 93.4 mm
- net Net-(U1--): track 0.00 -> 48.8 mm, vias 0 -> 2
- net +12V: track 0.00 -> 37.9 mm
- net -12V: track 0.00 -> 36.3 mm
- net GND: track 0.00 -> 31.5 mm
- net Net-(C6-Pad1): track 0.00 -> 26.0 mm
- net Net-(C3-Pad1): track 0.00 -> 18.1 mm
- net Net-(C1-Pad1): track 0.00 -> 15.6 mm
- net Signal_INPUT: track 0.00 -> 13.3 mm
- net Net-(C7-Pad2): track 0.00 -> 12.3 mm
- net Net-(U1-+): track 0.00 -> 8.71 mm
- net Net-(C4-Pad1): track 0.00 -> 2.05 mm
- added copper zone on B.Cu, net -12V
